Commit message: [Add] warehouse_ground

File: ssapang_ws/src/turtlebot3_description/urdf/turtlebot3_burger.gazebo.xacro (robot description, xacro)
@@ -168,8 +168,8 @@
           <horizontal_fov>1.085595</horizontal_fov>
           <image>
-              <!-- <width>640</width> -->
-              <!-- <height>480</height> -->
-              <width>480</width>
-              <height>640</height>
+              <width>640</width>
+              <height>480</height>
+              <!-- <width>480</width> -->
+              <!-- <height>640</height> -->
               <format>R8G8B8</format>
           </image>

File: ssapang_ws/src/turtlebot3_description/urdf/turtlebot3_burger.urdf.xacro (robot description, xacro)
@@ -170,5 +170,5 @@
   <joint name="camera_joint2" type="fixed">
     <!-- <origin xyz="0.073 -0.011 0.084" rpy="0 0 0"/> -->
-    <origin xyz="0.073 -0.011 1.084" rpy="0 0 0"/>
+    <origin xyz="0.073 -0.011 0.184" rpy="0 -60 0"/>
     <parent link="base_link"/>
     <child link="camera_link2"/>
