Commit message: [FEAT] multi-robot spawn(not multi-rrbot)

File: ssapang_ws/src/ssabot/urdf/turtlebot3_waffle.gazebo.xacro (robot description, xacro)
@@ -4,4 +4,11 @@
   <xacro:arg name="camera_visual" default="false"/>
   <xacro:arg name="imu_visual"    default="false"/>
+  <!-- Add gazebo_ros_control plugin -->
+  <gazebo>
+    <plugin name="gazebo_ros_control" filename="libgazebo_ros_control.so">
+      <robotNamespace>/waffle</robotNamespace>
+      <robotSimType>gazebo_ros_control/DefaultRobotHWSim</robotSimType>
+    </plugin>
+  </gazebo>
   <gazebo reference="base_link">
     <material>Gazebo/DarkGrey</material>

File: ssapang_ws/src/ssabot/urdf/turtlebot3_waffle.urdf.xacro (robot description, xacro)
@@ -1,6 +1,6 @@
 <?xml version="1.0" ?>
 <robot name="turtlebot3_waffle" xmlns:xacro="http://ros.org/wiki/xacro">
-  <xacro:include filename="$(find turtlebot3_description)/urdf/common_properties.xacro"/>
-  <xacro:include filename="$(find turtlebot3_description)/urdf/turtlebot3_waffle.gazebo.xacro"/>
+  <xacro:include filename="$(find ssabot)/urdf/common_properties.xacro"/>
+  <xacro:include filename="$(find ssabot)/urdf/turtlebot3_waffle.gazebo.xacro"/>
   <xacro:property name="r200_cam_rgb_px" value="0.005"/>
   <xacro:property name="r200_cam_rgb_py" value="0.018"/>
@@ -17,5 +17,5 @@
       <origin xyz="-0.064 0 0.0" rpy="0 0 0"/>
       <geometry>
-        <mesh filename="package://turtlebot3_description/meshes/bases/waffle_base.stl" scale="0.001 0.001 0.001"/>
+        <mesh filename="package://ssabot/meshes/bases/waffle_base.stl" scale="0.001 0.001 0.001"/>
       </geometry>
       <material name="light_black"/>
@@ -65,5 +65,5 @@
     <origin xyz="0 0 0" rpy="0 0 0"/>
     <axis xyz="0 0 1"/>
-    <limit effort="30" lower="-0.01" upper="0.01" velocity="1.571"/>
+    <limit effort="30" lower="-0.1" upper="0.1" velocity="0.171"/>
   </joint>
   <link name="piston_link2">
@@ -89,15 +89,15 @@
       <origin xyz="-0.05 0 0.17" rpy="0 0 1.57"/>
       <geometry>
-        <mesh filename="package://turtlebot3_description/meshes/piston/piston_plate.stl" scale="0.015 0.015 0.015"/>
+        <mesh filename="package://ssabot/meshes/piston/piston_plate.dae" scale="0.015 0.015 0.015"/>
       </geometry>
       <material name="dark"/>
     </visual>
+    <collision>
+      <origin xyz="-0.05 0 0.17" rpy="0 0 1.57"/>
+      <geometry>
+        <mesh filename="package://ssabot/meshes/piston/piston_plate.dae" scale="0.015 0.015 0.015"/>
+      </geometry>
+    </collision>
 <!--
-    <collision>
-      <origin xyz="0.015 0 -0.0065" rpy="0 0 0"/>
-      <geometry>
-        <cylinder length="0.0315" radius="0.055"/>
-      </geometry>
-    </collision>
     <inertial>
       <mass value="0.114" />
@@ -108,30 +108,14 @@
     </inertial> -->
   </link>
-  <!-- <joint name="fixed" type="fixed">
-    <parent link="link1"/>
-    <child link="link2"/>
-  </joint>
-  <link name="link3">
-    <collision>
-      <origin xyz="0 0 1" rpy="0 1.57 0"/>
-      <geometry>
-        <cylinder length="2" radius="0.1"/>
-      </geometry>
-    </collision>
-    <visual>
-      <origin xyz="0 0 1" rpy= "0 1.57 0"/>
-      <geometry>
-        <cylinder length="2" radius="0.1"/>
-      </geometry>
-      <material name="red">
-          <color rgba="1 0 0 1"/>
-      </material>
-    </visual>
-    <inertial>
-      <origin xyz="0 0 0" rpy="0 0 0"/>
-      <mass value="1"/>
-      <inertia ixx="1.0" ixy="0.0" ixz="0.0" iyy="1.0" iyz="0.0" izz="1.0"/>
-    </inertial>
-  </link> -->
+  <transmission name="waffle_tran">
+    <type>transmission_interface/SimpleTransmission</type>
+    <joint name="piston_joint2">
+      <hardwareInterface>hardware_interface/PositionJointInterface</hardwareInterface>
+    </joint>
+    <actuator name="waffle_motor">
+      <hardwareInterface>hardware_interface/PositionJointInterface</hardwareInterface>
+      <mechanicalReduction>1</mechanicalReduction>
+    </actuator>
+  </transmission>
   <!---->
   <joint name="wheel_left_joint" type="continuous">
@@ -145,5 +129,5 @@
       <origin xyz="0 0 0" rpy="1.57 0 0"/>
       <geometry>
-        <mesh filename="package://turtlebot3_description/meshes/wheels/left_tire.stl" scale="0.001 0.001 0.001"/>
+        <mesh filename="package://ssabot/meshes/wheels/left_tire.stl" scale="0.001 0.001 0.001"/>
       </geometry>
       <material name="dark"/>
@@ -173,5 +157,5 @@
       <origin xyz="0 0 0" rpy="1.57 0 0"/>
       <geometry>
-        <mesh filename="package://turtlebot3_description/meshes/wheels/right_tire.stl" scale="0.001 0.001 0.001"/>
+        <mesh filename="package://ssabot/meshes/wheels/right_tire.stl" scale="0.001 0.001 0.001"/>
       </geometry>
       <material name="dark"/>
@@ -246,5 +230,5 @@
       <origin xyz="0 0 0" rpy="0 0 0"/>
       <geometry>
-        <mesh filename="package://turtlebot3_description/meshes/sensors/lds.stl" scale="0.001 0.001 0.001"/>
+        <mesh filename="package://ssabot/meshes/sensors/lds.stl" scale="0.001 0.001 0.001"/>
       </geometry>
       <material name="dark"/>
@@ -273,5 +257,5 @@
      <origin xyz="0 0 0" rpy="1.57 0 1.57"/>
       <geometry>
-       <mesh filename="package://turtlebot3_description/meshes/sensors/r200.dae" />
+       <mesh filename="package://ssabot/meshes/sensors/r200.dae" />
       </geometry>
     </visual>

Commit message: [Feat] add push robot example

File: ssapang_ws/src/ssabot/urdf/turtlebot3_waffle.gazebo.xacro (robot description, xacro)
@@ -11,5 +11,5 @@
   </gazebo>
   <gazebo reference="base_link">
-    <material>Gazebo/DarkGrey</material>
+    <material>Gazebo/White</material>
   </gazebo>
   <gazebo reference="wheel_left_link">

Commit message: [modified] control tower

File: ssapang_ws/src/ssabot/urdf/turtlebot3_waffle.gazebo.xacro (robot description, xacro)
@@ -108,5 +108,5 @@
     </plugin>
   </gazebo>
-  <gazebo reference="base_scan">
+  <!-- <gazebo reference="base_scan">
     <material>Gazebo/FlatBlack</material>
     <sensor type="ray" name="lds_lfcd_sensor">
@@ -139,5 +139,5 @@
       </plugin>
     </sensor>
-  </gazebo>
+  </gazebo> -->
   <gazebo reference="camera_rgb_frame">
     <sensor type="depth" name="realsense_R200">

File: ssapang_ws/src/ssabot/urdf/turtlebot3_waffle.urdf.xacro (robot description, xacro)
@@ -36,17 +36,17 @@
   </link>
   <!-- Add piston plate-->
-  <joint name="piston_joint1" type="fixed">
+  <!-- <joint name="piston_joint1" type="fixed">
     <parent link="base_link"/>
     <child link="piston_link1"/>
   </joint>
   <link name="piston_link1">
-    <!-- <collision>
+    <collision>
       <origin xyz="0 -0.004 0.015" rpy="0 0 0"/>
       <geometry>
         <cylinder length="0.02" radius="0.005"/>
       </geometry>
-    </collision> -->
-    <visual>
-      <origin xyz="-0.05 0 0.14" rpy="0 0 0"/>
+    </collision>
+    <visual>
+	  <origin xyz="-0.05 0 0.14" rpy="0 0 0"/>
       <geometry>
         <cylinder length="0.02" radius="0.005"/>
@@ -56,5 +56,5 @@
     <inertial>
       <origin xyz="0 0 0" rpy="0 0 0"/>
-      <mass value="0.001"/>
+      <mass value="0.00001"/>
       <inertia ixx="0.0" ixy="0.0" ixz="0.0" iyy="0.0" iyz="0.0" izz="0.0"/>
     </inertial>
@@ -69,5 +69,5 @@
   <link name="piston_link2">
     <visual>
-      <origin xyz="-0.05 0 0.16" rpy="0 0 0"/>
+	  <origin xyz="-0.05 0 0.16" rpy="0 0 0"/>
       <geometry>
         <cylinder length="0.02" radius="0.01"/>
@@ -77,6 +77,6 @@
     <inertial>
       <origin xyz="0 0 0" rpy="0 0 0"/>
-      <mass value="0.001"/>
-      <inertia ixx="0.0" ixy="0.0" ixz="0.0" iyy="0.0" iyz="0.0" izz="0.0"/>
+      <mass value="0.00001"/>
+      <inertia ixx="0.0" ixy="0.0" ixz="0." iyy="0.0" iyz="0.0" izz="0.0"/>
     </inertial>
   </link>
@@ -98,13 +98,12 @@
         <mesh filename="package://ssabot/meshes/piston/piston_plate.dae" scale="0.015 0.015 0.015"/>
       </geometry>
-    </collision>
-<!--
-    <inertial>
-      <mass value="0.114" />
-      <origin xyz="0 0 0" />
-      <inertia ixx="0.001" ixy="0.0" ixz="0.0"
-               iyy="0.001" iyz="0.0"
-               izz="0.001" />
-    </inertial> -->
+      </collision>
+          <inertial>
+            <mass value="0.114" />
+            <origin xyz="0 0 0" />
+            <inertia ixx="0.001" ixy="0.0" ixz="0.0"
+                    iyy="0.001" iyz="0.0"
+                    izz="0.001" />
+          </inertial>
   </link>
   <transmission name="waffle_tran">
@@ -117,5 +116,5 @@
       <mechanicalReduction>1</mechanicalReduction>
     </actuator>
-  </transmission>
+  </transmission> -->
   <!---->
   <joint name="wheel_left_joint" type="continuous">
@@ -221,5 +220,5 @@
   </joint>
   <link name="imu_link"/>
-  <joint name="scan_joint" type="fixed">
+  <!-- <joint name="scan_joint" type="fixed">
     <parent link="base_link"/>
     <child link="base_scan"/>
@@ -247,55 +246,4 @@
                izz="0.001" />
     </inertial>
-  </link>
-  <joint name="camera_joint" type="fixed">
-    <origin xyz="0.064 -0.065 0.094" rpy="0 0 0"/>
-    <parent link="base_link"/>
-    <child link="camera_link"/>
-  </joint>
-  <link name="camera_link">
-    <visual>
-     <origin xyz="0 0 0" rpy="1.57 0 1.57"/>
-      <geometry>
-       <mesh filename="package://ssabot/meshes/sensors/r200.dae" />
-      </geometry>
-    </visual>
-    <collision>
-      <origin xyz="0.003 0.065 0.007" rpy="0 0 0"/>
-      <geometry>
-        <box size="0.012 0.132 0.020"/>
-      </geometry>
-    </collision>
-    <!-- This inertial field needs doesn't contain reliable data!! -->
-<!--   <inertial>
-      <mass value="0.564" />
-      <origin xyz="0 0 0" />
-      <inertia ixx="0.003881243" ixy="0.0" ixz="0.0"
-               iyy="0.000498940" iyz="0.0"
-               izz="0.003879257" />
-    </inertial>-->
-  </link>
-  <joint name="camera_rgb_joint" type="fixed">
-    <origin xyz="${r200_cam_rgb_px} ${r200_cam_rgb_py} ${r200_cam_rgb_pz}" rpy="0 0 0"/>
-    <parent link="camera_link"/>
-    <child link="camera_rgb_frame"/>
-  </joint>
-  <link name="camera_rgb_frame"/>
-  <joint name="camera_rgb_optical_joint" type="fixed">
-    <origin xyz="0 0 0" rpy="-1.57 0 -1.57"/>
-    <parent link="camera_rgb_frame"/>
-    <child link="camera_rgb_optical_frame"/>
-  </joint>
-  <link name="camera_rgb_optical_frame"/>
-  <joint name="camera_depth_joint" type="fixed">
-    <origin xyz="${r200_cam_rgb_px} ${r200_cam_rgb_py + r200_cam_depth_offset} ${r200_cam_rgb_pz}" rpy="0 0 0"/>
-    <parent link="camera_link"/>
-    <child link="camera_depth_frame"/>
-  </joint>
-  <link name="camera_depth_frame"/>
-  <joint name="camera_depth_optical_joint" type="fixed">
-    <origin xyz="0 0 0" rpy="-1.57 0 -1.57"/>
-    <parent link="camera_depth_frame"/>
-    <child link="camera_depth_optical_frame"/>
-  </joint>
-  <link name="camera_depth_optical_frame"/>
+  </link> -->
 </robot>
