Commit message: [Modified] control code

File: ssapang_ws/src/ssabot/urdf/turtlebot3_burger.gazebo.xacro (robot description, xacro)
@@ -126,5 +126,5 @@
   </gazebo>
   <!-- add waffle_pi camera -->
-  <gazebo reference="camera_rgb_frame">
+  <!-- <gazebo reference="camera_rgb_frame">
     <sensor type="camera" name="Pi Camera">
       <always_on>true</always_on>
@@ -135,6 +135,4 @@
               <width>640</width>
               <height>480</height>
-              <!-- <width>480</width> -->
-              <!-- <height>640</height> -->
               <format>R8G8B8</format>
           </image>
@@ -159,7 +157,7 @@
       </plugin>
     </sensor>
-  </gazebo>
+  </gazebo> -->
   <!-- add second camera -->
-  <gazebo reference="camera_rgb_frame2">
+  <!-- <gazebo reference="camera_rgb_frame2">
     <sensor type="camera" name="Pi Camera">
       <always_on>true</always_on>
@@ -168,6 +166,4 @@
           <horizontal_fov>1.085595</horizontal_fov>
           <image>
-              <!-- <width>640</width> -->
-              <!-- <height>480</height> -->
               <width>480</width>
               <height>640</height>
@@ -194,4 +190,4 @@
       </plugin>
     </sensor>
-  </gazebo>
+  </gazebo> -->
 </robot>

File: ssapang_ws/src/ssabot/urdf/turtlebot3_burger.urdf.xacro (robot description, xacro)
@@ -141,7 +141,6 @@
   </link>
 <!-- add waffle_pi camera -->
-  <joint name="camera_joint" type="fixed">
+  <!-- <joint name="camera_joint" type="fixed">
     <origin xyz="0.073 -0.011 0.084" rpy="0 0 0"/>
-    <!-- <origin xyz="0.073 -0.011 0.084" rpy="0 45 0"/> -->
     <parent link="base_link"/>
     <child link="camera_link"/>
@@ -166,8 +165,7 @@
     <child link="camera_rgb_optical_frame"/>
   </joint>
-  <link name="camera_rgb_optical_frame"/>
+  <link name="camera_rgb_optical_frame"/> -->
   <!-- add second camera -->
-  <joint name="camera_joint2" type="fixed">
-    <!-- <origin xyz="0.073 -0.011 0.084" rpy="0 0 0"/> -->
+  <!-- <joint name="camera_joint2" type="fixed">
     <origin xyz="0.073 -0.011 1.084" rpy="0 0 0"/>
     <parent link="base_link"/>
@@ -193,4 +191,4 @@
     <child link="camera_rgb_optical_frame2"/>
   </joint>
-  <link name="camera_rgb_optical_frame2"/>
+  <link name="camera_rgb_optical_frame2"/> -->
 </robot>

Commit message: [Modify]

File: ssapang_ws/src/ssabot/urdf/turtlebot3_burger.gazebo.xacro (robot description, xacro)
@@ -8,20 +8,20 @@
   </gazebo>
   <gazebo reference="wheel_left_link">
-    <mu1>0.1</mu1>
-    <mu2>0.1</mu2>
-    <kp>500000.0</kp>
-    <kd>10.0</kd>
+    <mu1>0.2</mu1>
+    <mu2>0.2</mu2>
+    <kp>1000000.0</kp>
+    <kd>20.0</kd>
     <minDepth>0.001</minDepth>
-    <maxVel>0.1</maxVel>
+    <maxVel>0.2</maxVel>
     <fdir1>1 0 0</fdir1>
     <material>Gazebo/FlatBlack</material>
   </gazebo>
   <gazebo reference="wheel_right_link">
-    <mu1>0.1</mu1>
-    <mu2>0.1</mu2>
-    <kp>500000.0</kp>
-    <kd>10.0</kd>
+    <mu1>0.2</mu1>
+    <mu2>0.2</mu2>
+    <kp>1000000.0</kp>
+    <kd>20.0</kd>
     <minDepth>0.001</minDepth>
-    <maxVel>0.1</maxVel>
+    <maxVel>0.2</maxVel>
     <fdir1>1 0 0</fdir1>
     <material>Gazebo/FlatBlack</material>
@@ -58,8 +58,8 @@
       <leftJoint>wheel_left_joint</leftJoint>
       <rightJoint>wheel_right_joint</rightJoint>
-      <wheelSeparation>0.160</wheelSeparation>
-      <wheelDiameter>0.066</wheelDiameter>
+      <wheelSeparation>0.320</wheelSeparation>
+      <wheelDiameter>0.132</wheelDiameter>
       <wheelAcceleration>1</wheelAcceleration>
-      <wheelTorque>10</wheelTorque>
+      <wheelTorque>15</wheelTorque>
       <rosDebugLevel>na</rosDebugLevel>
     </plugin>
@@ -124,4 +124,8 @@
       </plugin>
     </sensor>
+  </gazebo>
+  <!-- dump_box -->
+  <gazebo reference="dump_box_visual">
+    <material>Gazebo/Orange</material>
   </gazebo>
   <!-- add waffle_pi camera -->

File: ssapang_ws/src/ssabot/urdf/turtlebot3_burger.urdf.xacro (robot description, xacro)
@@ -7,18 +7,18 @@
     <parent link="base_footprint"/>
     <child link="base_link"/>
-    <origin xyz="0.0 0.0 0.010" rpy="0 0 0"/>
+    <origin xyz="0.0 0.0 0.020" rpy="0 0 0"/>
   </joint>
   <link name="base_link">
     <visual>
-      <origin xyz="-0.032 0 0.0" rpy="0 0 0"/>
-      <geometry>
-        <mesh filename="package://ssabot/meshes/bases/burger_base.stl" scale="0.001 0.001 0.001"/>
+      <origin xyz="-0.064 0 0.0" rpy="0 0 0"/>
+      <geometry>
+        <mesh filename="package://ssabot/meshes/bases/burger_base.stl" scale="0.002 0.002 0.002"/>
       </geometry>
       <material name="light_black"/>
     </visual>
     <collision>
-      <origin xyz="-0.032 0 0.070" rpy="0 0 0"/>
-      <geometry>
-        <box size="0.140 0.140 0.143"/>
+      <origin xyz="-0.064 0 0.140" rpy="0 0 0"/>
+      <geometry>
+        <box size="0.280 0.280 0.286"/>
       </geometry>
     </collision>
@@ -34,5 +34,5 @@
     <parent link="base_link"/>
     <child link="wheel_left_link"/>
-    <origin xyz="0.0 0.08 0.023" rpy="-1.57 0 0"/>
+    <origin xyz="0.0 0.16 0.046" rpy="-1.57 0 0"/>
     <axis xyz="0 0 1"/>
   </joint>
@@ -41,5 +41,5 @@
       <origin xyz="0 0 0" rpy="1.57 0 0"/>
       <geometry>
-        <mesh filename="package://ssabot/meshes/wheels/left_tire.stl" scale="0.001 0.001 0.001"/>
+        <mesh filename="package://ssabot/meshes/wheels/left_tire.stl" scale="0.002 0.002 0.002"/>
       </geometry>
       <material name="dark"/>
@@ -48,13 +48,13 @@
       <origin xyz="0 0 0" rpy="0 0 0"/>
       <geometry>
-        <cylinder length="0.018" radius="0.033"/>
-      </geometry>
-    </collision>
-    <inertial>
-      <origin xyz="0 0 0" />
-      <mass value="2.8498940e-02" />
-      <inertia ixx="1.1175580e-05" ixy="-4.2369783e-11" ixz="-5.9381719e-09"
-               iyy="1.1192413e-05" iyz="-1.4400107e-11"
-               izz="2.0712558e-05" />
+        <cylinder length="0.036" radius="0.066"/>
+      </geometry>
+    </collision>
+    <inertial>
+      <origin xyz="0 0 0" />
+      <mass value="5.6398940e-02" />
+      <inertia ixx="2.1175580e-05" ixy="-8.2369783e-11" ixz="-10.9381719e-09"
+               iyy="2.1192413e-05" iyz="-2.4400107e-11"
+               izz="4.0712558e-05" />
       </inertial>
   </link>
@@ -62,5 +62,5 @@
     <parent link="base_link"/>
     <child link="wheel_right_link"/>
-    <origin xyz="0.0 -0.080 0.023" rpy="-1.57 0 0"/>
+    <origin xyz="0.0 -0.160 0.046" rpy="-1.57 0 0"/>
     <axis xyz="0 0 1"/>
   </joint>
@@ -69,5 +69,5 @@
       <origin xyz="0 0 0" rpy="1.57 0 0"/>
       <geometry>
-        <mesh filename="package://ssabot/meshes/wheels/right_tire.stl" scale="0.001 0.001 0.001"/>
+        <mesh filename="package://ssabot/meshes/wheels/right_tire.stl" scale="0.002 0.002 0.002"/>
       </geometry>
       <material name="dark"/>
@@ -76,13 +76,13 @@
       <origin xyz="0 0 0" rpy="0 0 0"/>
       <geometry>
-        <cylinder length="0.018" radius="0.033"/>
-      </geometry>
-    </collision>
-    <inertial>
-      <origin xyz="0 0 0" />
-      <mass value="2.8498940e-02" />
-      <inertia ixx="1.1175580e-05" ixy="-4.2369783e-11" ixz="-5.9381719e-09"
-               iyy="1.1192413e-05" iyz="-1.4400107e-11"
-               izz="2.0712558e-05" />
+        <cylinder length="0.036" radius="0.066"/>
+      </geometry>
+    </collision>
+    <inertial>
+      <origin xyz="0 0 0" />
+      <mass value="5.6398940e-02" />
+      <inertia ixx="2.1175580e-05" ixy="-8.2369783e-11" ixz="-10.9381719e-09"
+               iyy="2.1192413e-05" iyz="-2.4400107e-11"
+               izz="4.0712558e-05" />
       </inertial>
   </link>
@@ -90,19 +90,19 @@
     <parent link="base_link"/>
     <child link="caster_back_link"/>
-    <origin xyz="-0.081 0 -0.004" rpy="-1.57 0 0"/>
+    <origin xyz="-0.162 0 -0.008" rpy="-1.57 0 0"/>
   </joint>
   <link name="caster_back_link">
     <collision>
-      <origin xyz="0 0.001 0" rpy="0 0 0"/>
-      <geometry>
-        <box size="0.030 0.009 0.020"/>
-      </geometry>
-    </collision>
-    <inertial>
-      <origin xyz="0 0 0" />
-      <mass value="0.005" />
-      <inertia ixx="0.001" ixy="0.0" ixz="0.0"
-               iyy="0.001" iyz="0.0"
-               izz="0.001" />
+      <origin xyz="0 0.002 0" rpy="0 0 0"/>
+      <geometry>
+        <box size="0.060 0.018 0.040"/>
+      </geometry>
+    </collision>
+    <inertial>
+      <origin xyz="0 0 0" />
+      <mass value="0.010" />
+      <inertia ixx="0.002" ixy="0.0" ixz="0.0"
+               iyy="0.002" iyz="0.0"
+               izz="0.002" />
     </inertial>
   </link>
@@ -116,8 +116,8 @@
     <parent link="base_link"/>
     <child link="base_scan"/>
-    <origin xyz="-0.032 0 0.172" rpy="0 0 0"/>
+    <origin xyz="0 0 0.28" rpy="0 0 0"/>
   </joint>
   <link name="base_scan">
-    <visual>
+    <!-- <visual>
       <origin xyz="0 0 0.0" rpy="0 0 0"/>
       <geometry>
@@ -131,7 +131,19 @@
         <cylinder length="0.0315" radius="0.055"/>
       </geometry>
-    </collision>
-    <inertial>
-      <mass value="0.114" />
+    </collision> -->
+    <collision name='collision'>
+      <origin xyz="0 0 0" rpy=" 0 0 0"/>
+        <geometry>
+          <mesh filename="package://ssabot/meshes/meshes/dumper_bin.dae" scale="0.015 0.015 0.015"/>
+        </geometry>
+    </collision>
+    <visual name='dump_box_visual'>
+      <origin xyz=" 0 0 0.0" rpy="0 0 1.57079"/>
+        <geometry>
+          <mesh filename="package://ssabot/meshes/meshes/dumper_bin.dae" scale="0.015 0.015 0.015"/>
+        </geometry>
+    </visual>
+    <inertial>
+      <mass value="0.01" />
       <origin xyz="0 0 0" />
       <inertia ixx="0.001" ixy="0.0" ixz="0.0"

Commit message: [modified] control tower

File: ssapang_ws/src/ssabot/urdf/turtlebot3_burger.gazebo.xacro (robot description, xacro)
@@ -8,20 +8,20 @@
   </gazebo>
   <gazebo reference="wheel_left_link">
-    <mu1>0.1</mu1>
-    <mu2>0.1</mu2>
-    <kp>500000.0</kp>
-    <kd>10.0</kd>
+    <mu1>0.2</mu1>
+    <mu2>0.2</mu2>
+    <kp>1000000.0</kp>
+    <kd>20.0</kd>
     <minDepth>0.001</minDepth>
-    <maxVel>0.1</maxVel>
+    <maxVel>0.2</maxVel>
     <fdir1>1 0 0</fdir1>
     <material>Gazebo/FlatBlack</material>
   </gazebo>
   <gazebo reference="wheel_right_link">
-    <mu1>0.1</mu1>
-    <mu2>0.1</mu2>
-    <kp>500000.0</kp>
-    <kd>10.0</kd>
+    <mu1>0.2</mu1>
+    <mu2>0.2</mu2>
+    <kp>1000000.0</kp>
+    <kd>20.0</kd>
     <minDepth>0.001</minDepth>
-    <maxVel>0.1</maxVel>
+    <maxVel>0.2</maxVel>
     <fdir1>1 0 0</fdir1>
     <material>Gazebo/FlatBlack</material>
@@ -58,8 +58,8 @@
       <leftJoint>wheel_left_joint</leftJoint>
       <rightJoint>wheel_right_joint</rightJoint>
-      <wheelSeparation>0.160</wheelSeparation>
-      <wheelDiameter>0.066</wheelDiameter>
+      <wheelSeparation>0.320</wheelSeparation>
+      <wheelDiameter>0.132</wheelDiameter>
       <wheelAcceleration>1</wheelAcceleration>
-      <wheelTorque>10</wheelTorque>
+      <wheelTorque>15</wheelTorque>
       <rosDebugLevel>na</rosDebugLevel>
     </plugin>
@@ -124,4 +124,8 @@
       </plugin>
     </sensor>
+  </gazebo>
+  <!-- dump_box -->
+  <gazebo reference="dump_box_visual">
+    <material>Gazebo/Orange</material>
   </gazebo>
   <!-- add waffle_pi camera -->

File: ssapang_ws/src/ssabot/urdf/turtlebot3_burger.urdf.xacro (robot description, xacro)
@@ -7,18 +7,18 @@
     <parent link="base_footprint"/>
     <child link="base_link"/>
-    <origin xyz="0.0 0.0 0.010" rpy="0 0 0"/>
+    <origin xyz="0.0 0.0 0.020" rpy="0 0 0"/>
   </joint>
   <link name="base_link">
     <visual>
-      <origin xyz="-0.032 0 0.0" rpy="0 0 0"/>
-      <geometry>
-        <mesh filename="package://ssabot/meshes/bases/burger_base.stl" scale="0.001 0.001 0.001"/>
+      <origin xyz="-0.064 0 0.0" rpy="0 0 0"/>
+      <geometry>
+        <mesh filename="package://ssabot/meshes/bases/burger_base.stl" scale="0.002 0.002 0.002"/>
       </geometry>
       <material name="light_black"/>
     </visual>
     <collision>
-      <origin xyz="-0.032 0 0.070" rpy="0 0 0"/>
-      <geometry>
-        <box size="0.140 0.140 0.143"/>
+      <origin xyz="-0.064 0 0.140" rpy="0 0 0"/>
+      <geometry>
+        <box size="0.280 0.280 0.286"/>
       </geometry>
     </collision>
@@ -34,5 +34,5 @@
     <parent link="base_link"/>
     <child link="wheel_left_link"/>
-    <origin xyz="0.0 0.08 0.023" rpy="-1.57 0 0"/>
+    <origin xyz="0.0 0.16 0.046" rpy="-1.57 0 0"/>
     <axis xyz="0 0 1"/>
   </joint>
@@ -41,5 +41,5 @@
       <origin xyz="0 0 0" rpy="1.57 0 0"/>
       <geometry>
-        <mesh filename="package://ssabot/meshes/wheels/left_tire.stl" scale="0.001 0.001 0.001"/>
+        <mesh filename="package://ssabot/meshes/wheels/left_tire.stl" scale="0.002 0.002 0.002"/>
       </geometry>
       <material name="dark"/>
@@ -48,13 +48,13 @@
       <origin xyz="0 0 0" rpy="0 0 0"/>
       <geometry>
-        <cylinder length="0.018" radius="0.033"/>
-      </geometry>
-    </collision>
-    <inertial>
-      <origin xyz="0 0 0" />
-      <mass value="2.8498940e-02" />
-      <inertia ixx="1.1175580e-05" ixy="-4.2369783e-11" ixz="-5.9381719e-09"
-               iyy="1.1192413e-05" iyz="-1.4400107e-11"
-               izz="2.0712558e-05" />
+        <cylinder length="0.036" radius="0.066"/>
+      </geometry>
+    </collision>
+    <inertial>
+      <origin xyz="0 0 0" />
+      <mass value="5.6398940e-02" />
+      <inertia ixx="2.1175580e-05" ixy="-8.2369783e-11" ixz="-10.9381719e-09"
+               iyy="2.1192413e-05" iyz="-2.4400107e-11"
+               izz="4.0712558e-05" />
       </inertial>
   </link>
@@ -62,5 +62,5 @@
     <parent link="base_link"/>
     <child link="wheel_right_link"/>
-    <origin xyz="0.0 -0.080 0.023" rpy="-1.57 0 0"/>
+    <origin xyz="0.0 -0.160 0.046" rpy="-1.57 0 0"/>
     <axis xyz="0 0 1"/>
   </joint>
@@ -69,5 +69,5 @@
       <origin xyz="0 0 0" rpy="1.57 0 0"/>
       <geometry>
-        <mesh filename="package://ssabot/meshes/wheels/right_tire.stl" scale="0.001 0.001 0.001"/>
+        <mesh filename="package://ssabot/meshes/wheels/right_tire.stl" scale="0.002 0.002 0.002"/>
       </geometry>
       <material name="dark"/>
@@ -76,13 +76,13 @@
       <origin xyz="0 0 0" rpy="0 0 0"/>
       <geometry>
-        <cylinder length="0.018" radius="0.033"/>
-      </geometry>
-    </collision>
-    <inertial>
-      <origin xyz="0 0 0" />
-      <mass value="2.8498940e-02" />
-      <inertia ixx="1.1175580e-05" ixy="-4.2369783e-11" ixz="-5.9381719e-09"
-               iyy="1.1192413e-05" iyz="-1.4400107e-11"
-               izz="2.0712558e-05" />
+        <cylinder length="0.036" radius="0.066"/>
+      </geometry>
+    </collision>
+    <inertial>
+      <origin xyz="0 0 0" />
+      <mass value="5.6398940e-02" />
+      <inertia ixx="2.1175580e-05" ixy="-8.2369783e-11" ixz="-10.9381719e-09"
+               iyy="2.1192413e-05" iyz="-2.4400107e-11"
+               izz="4.0712558e-05" />
       </inertial>
   </link>
@@ -90,19 +90,19 @@
     <parent link="base_link"/>
     <child link="caster_back_link"/>
-    <origin xyz="-0.081 0 -0.004" rpy="-1.57 0 0"/>
+    <origin xyz="-0.162 0 -0.008" rpy="-1.57 0 0"/>
   </joint>
   <link name="caster_back_link">
     <collision>
-      <origin xyz="0 0.001 0" rpy="0 0 0"/>
-      <geometry>
-        <box size="0.030 0.009 0.020"/>
-      </geometry>
-    </collision>
-    <inertial>
-      <origin xyz="0 0 0" />
-      <mass value="0.005" />
-      <inertia ixx="0.001" ixy="0.0" ixz="0.0"
-               iyy="0.001" iyz="0.0"
-               izz="0.001" />
+      <origin xyz="0 0.002 0" rpy="0 0 0"/>
+      <geometry>
+        <box size="0.060 0.018 0.040"/>
+      </geometry>
+    </collision>
+    <inertial>
+      <origin xyz="0 0 0" />
+      <mass value="0.010" />
+      <inertia ixx="0.002" ixy="0.0" ixz="0.0"
+               iyy="0.002" iyz="0.0"
+               izz="0.002" />
     </inertial>
   </link>
@@ -116,8 +116,8 @@
     <parent link="base_link"/>
     <child link="base_scan"/>
-    <origin xyz="-0.032 0 0.172" rpy="0 0 0"/>
+    <origin xyz="0 0 0.28" rpy="0 0 0"/>
   </joint>
   <link name="base_scan">
-    <visual>
+    <!-- <visual>
       <origin xyz="0 0 0.0" rpy="0 0 0"/>
       <geometry>
@@ -131,7 +131,19 @@
         <cylinder length="0.0315" radius="0.055"/>
       </geometry>
-    </collision>
-    <inertial>
-      <mass value="0.114" />
+    </collision> -->
+    <collision name='collision'>
+      <origin xyz="0 0 0" rpy=" 0 0 0"/>
+        <geometry>
+          <mesh filename="package://ssabot/meshes/meshes/dumper_bin.dae" scale="0.01 0.01 0.01"/>
+        </geometry>
+    </collision>
+    <visual name='dump_box_visual'>
+      <origin xyz=" 0 0 0.0" rpy="0 0 1.57079"/>
+        <geometry>
+          <mesh filename="package://ssabot/meshes/meshes/dumper_bin.dae" scale="0.01 0.01 0.01"/>
+        </geometry>
+    </visual>
+    <inertial>
+      <mass value="0.01" />
       <origin xyz="0 0 0" />
       <inertia ixx="0.001" ixy="0.0" ixz="0.0"

File: ssapang_ws/src/ssabot/urdf/turtlebot3_waffle.gazebo.xacro (robot description, xacro)
@@ -76,5 +76,5 @@
       <wheelDiameter>0.066</wheelDiameter>
       <wheelAcceleration>1</wheelAcceleration>
-      <wheelTorque>10</wheelTorque>
+      <wheelTorque>20</wheelTorque>
       <rosDebugLevel>na</rosDebugLevel>
     </plugin>
@@ -108,5 +108,5 @@
     </plugin>
   </gazebo>
-  <!-- <gazebo reference="base_scan">
+  <gazebo reference="base_scan">
     <material>Gazebo/FlatBlack</material>
     <sensor type="ray" name="lds_lfcd_sensor">
@@ -139,47 +139,11 @@
       </plugin>
     </sensor>
-  </gazebo> -->
-  <gazebo reference="camera_rgb_frame">
-    <sensor type="depth" name="realsense_R200">
-      <always_on>true</always_on>
-      <visualize>$(arg camera_visual)</visualize>
-      <camera>
-          <horizontal_fov>1.3439</horizontal_fov>
-          <image>
-              <width>1920</width>
-              <height>1080</height>
-              <format>R8G8B8</format>
-          </image>
-          <depth_camera></depth_camera>
-          <clip>
-              <near>0.03</near>
-              <far>100</far>
-          </clip>
-      </camera>
-      <plugin name="camera_controller" filename="libgazebo_ros_openni_kinect.so">
-        <baseline>0.2</baseline>
-        <alwaysOn>true</alwaysOn>
-        <updateRate>30.0</updateRate>
-        <cameraName>camera</cameraName>
-        <frameName>camera_rgb_optical_frame</frameName>
-        <imageTopicName>rgb/image_raw</imageTopicName>
-        <depthImageTopicName>depth/image_raw</depthImageTopicName>
-        <pointCloudTopicName>depth/points</pointCloudTopicName>
-        <cameraInfoTopicName>rgb/camera_info</cameraInfoTopicName>
-        <depthImageCameraInfoTopicName>depth/camera_info</depthImageCameraInfoTopicName>
-        <pointCloudCutoff>0.4</pointCloudCutoff>
-            <hackBaseline>0.07</hackBaseline>
-            <distortionK1>0.0</distortionK1>
-            <distortionK2>0.0</distortionK2>
-            <distortionK3>0.0</distortionK3>
-            <distortionT1>0.0</distortionT1>
-            <distortionT2>0.0</distortionT2>
-        <CxPrime>0.0</CxPrime>
-        <Cx>0.0</Cx>
-        <Cy>0.0</Cy>
-        <focalLength>0</focalLength>
-        <hackBaseline>0</hackBaseline>
-      </plugin>
-    </sensor>
+  </gazebo>
+  <gazebo reference="piston_plate">
+    <mu1>1</mu1>
+    <mu2>1</mu2>
+    <kp>1000000.0</kp>
+    <kd>10000.0</kd>
+    <material>Gazebo/FlatBlack</material>
   </gazebo>
 </robot>

File: ssapang_ws/src/ssabot/urdf/turtlebot3_waffle.urdf.xacro (robot description, xacro)
@@ -36,17 +36,17 @@
   </link>
   <!-- Add piston plate-->
-  <!-- <joint name="piston_joint1" type="fixed">
+  <joint name="piston_joint1" type="fixed">
     <parent link="base_link"/>
     <child link="piston_link1"/>
   </joint>
   <link name="piston_link1">
-    <collision>
+    <!-- <collision>
       <origin xyz="0 -0.004 0.015" rpy="0 0 0"/>
       <geometry>
         <cylinder length="0.02" radius="0.005"/>
       </geometry>
-    </collision>
-    <visual>
-	  <origin xyz="-0.05 0 0.14" rpy="0 0 0"/>
+    </collision> -->
+    <visual>
+      <origin xyz="-0.05 0 0.14" rpy="0 0 0"/>
       <geometry>
         <cylinder length="0.02" radius="0.005"/>
@@ -56,5 +56,5 @@
     <inertial>
       <origin xyz="0 0 0" rpy="0 0 0"/>
-      <mass value="0.00001"/>
+      <mass value="0.001"/>
       <inertia ixx="0.0" ixy="0.0" ixz="0.0" iyy="0.0" iyz="0.0" izz="0.0"/>
     </inertial>
@@ -65,9 +65,9 @@
     <origin xyz="0 0 0" rpy="0 0 0"/>
     <axis xyz="0 0 1"/>
-    <limit effort="30" lower="-0.1" upper="0.1" velocity="0.171"/>
+    <limit effort="30" lower="-0.1" upper="0.3" velocity="0.171"/>
   </joint>
   <link name="piston_link2">
     <visual>
-	  <origin xyz="-0.05 0 0.16" rpy="0 0 0"/>
+      <origin xyz="-0.05 0 0.16" rpy="0 0 0"/>
       <geometry>
         <cylinder length="0.02" radius="0.01"/>
@@ -77,6 +77,6 @@
     <inertial>
       <origin xyz="0 0 0" rpy="0 0 0"/>
-      <mass value="0.00001"/>
-      <inertia ixx="0.0" ixy="0.0" ixz="0." iyy="0.0" iyz="0.0" izz="0.0"/>
+      <mass value="0.001"/>
+      <inertia ixx="0.0" ixy="0.0" ixz="0.0" iyy="0.0" iyz="0.0" izz="0.0"/>
     </inertial>
   </link>
@@ -87,23 +87,23 @@
   <link name="piston_plate">
     <visual>
-      <origin xyz="-0.05 0 0.17" rpy="0 0 1.57"/>
-      <geometry>
-        <mesh filename="package://ssabot/meshes/piston/piston_plate.dae" scale="0.015 0.015 0.015"/>
-      </geometry>
-      <material name="dark"/>
-    </visual>
-    <collision>
-      <origin xyz="-0.05 0 0.17" rpy="0 0 1.57"/>
-      <geometry>
-        <mesh filename="package://ssabot/meshes/piston/piston_plate.dae" scale="0.015 0.015 0.015"/>
-      </geometry>
-      </collision>
-          <inertial>
-            <mass value="0.114" />
-            <origin xyz="0 0 0" />
-            <inertia ixx="0.001" ixy="0.0" ixz="0.0"
-                    iyy="0.001" iyz="0.0"
-                    izz="0.001" />
-          </inertial>
+      <origin xyz="-0.064 0 0.17" rpy="0 0 1.57"/>
+      <geometry>
+        <mesh filename="package://ssabot/meshes/piston/untitled.dae" scale="0.005  0.005  0.01"/>
+      </geometry>
+      <material name="dark"/>
+    </visual>
+    <collision>
+      <origin xyz="-0.064 0 0.17" rpy="0 0 1.57"/>
+      <geometry>
+        <mesh filename="package://ssabot/meshes/piston/untitled.dae" scale="0.005  0.005 0.01"/>
+      </geometry>
+    </collision>
+    <inertial>
+      <mass value="0.114" />
+      <origin xyz="0 0 0" />
+      <inertia ixx="0.001" ixy="0.0" ixz="0.0"
+               iyy="0.001" iyz="0.0"
+               izz="0.001" />
+    </inertial>
   </link>
   <transmission name="waffle_tran">
@@ -116,5 +116,5 @@
       <mechanicalReduction>1</mechanicalReduction>
     </actuator>
-  </transmission> -->
+  </transmission>
   <!---->
   <joint name="wheel_left_joint" type="continuous">
@@ -220,5 +220,5 @@
   </joint>
   <link name="imu_link"/>
-  <!-- <joint name="scan_joint" type="fixed">
+  <joint name="scan_joint" type="fixed">
     <parent link="base_link"/>
     <child link="base_scan"/>
@@ -246,4 +246,4 @@
                izz="0.001" />
     </inertial>
-  </link> -->
+  </link>
 </robot>
