Commit message: [Add] Map

File: ssapang_ws/src/ssabot/urdf/turtlebot3_burger.gazebo.xacro (robot description, xacro)
@@ -4,4 +4,18 @@
   <xacro:arg name="imu_visual"   default="false"/>
   <xacro:arg name="camera_visual" default="false"/>
+  <transmission name="dump_bin_actuator">
+          <type>transmission_interface/SimpleTransmission</type>
+          <joint name="dump_joint">
+              <hardwareInterface>hardware_interface/EffortJointInterface</hardwareInterface>
+          </joint>
+          <actuator name="dump_motor">
+              <hardwareInterface>hardware_interface/EffortJointInterface</hardwareInterface>
+              <mechanicalReduction>1</mechanicalReduction>
+          </actuator>
+    </transmission>
+  <gazebo>
+    <plugin name="gazebo_ros_control" filename="libgazebo_ros_control.so">
+    </plugin>
+  </gazebo>
   <gazebo reference="base_link">
     <material>Gazebo/DarkGrey</material>

File: ssapang_ws/src/ssabot/urdf/turtlebot3_burger.urdf.xacro (robot description, xacro)
@@ -57,5 +57,5 @@
                iyy="2.1192413e-05" iyz="-2.4400107e-11"
                izz="4.0712558e-05" />
-      </inertial>
+    </inertial>
   </link>
   <joint name="wheel_right_joint" type="continuous">
@@ -113,37 +113,47 @@
   </joint>
   <link name="imu_link"/>
-  <joint name="scan_joint" type="fixed">
+  <joint name="dump_joint" type="revolute">
     <parent link="base_link"/>
-    <child link="base_scan"/>
-    <origin xyz="0 0 0.28" rpy="0 0 0"/>
+    <child link="dumper_bin"/>
+    <origin xyz="0.2 0 0.28" rpy="0 0 0"/>
+    <axis xyz="0 1 0"/>
+    <limit effort="1" velocity="1" lower="0" upper="0.6"/>
   </joint>
-  <link name="base_scan">
-    <!-- <visual>
-      <origin xyz="0 0 0.0" rpy="0 0 0"/>
-      <geometry>
-        <mesh filename="package://ssabot/meshes/sensors/lds.stl" scale="0.001 0.001 0.001"/>
-      </geometry>
-      <material name="dark"/>
-    </visual>
-    <collision>
-      <origin xyz="0.015 0 -0.0065" rpy="0 0 0"/>
-      <geometry>
-        <cylinder length="0.0315" radius="0.055"/>
-      </geometry>
-    </collision> -->
+  <!-- <link name="dumper_bin">
     <collision name='collision'>
-      <origin xyz="0 0 0" rpy=" 0 0 0"/>
+      <origin xyz="-0.15 0 0" rpy=" 0 0 1.57079"/>
         <geometry>
-          <mesh filename="package://ssabot/meshes/meshes/dumper_bin.dae" scale="0.01 0.01 0.01"/>
+          <box size="0.3 0.3 0.01"/>
         </geometry>
     </collision>
     <visual name='dump_box_visual'>
-      <origin xyz=" 0 0 0.0" rpy="0 0 1.57079"/>
+      <origin xyz=" -0.15 0 0.0" rpy="0 0 1.57079"/>
         <geometry>
-          <mesh filename="package://ssabot/meshes/meshes/dumper_bin.dae" scale="0.01 0.01 0.01"/>
+          <box size="0.3 0.3 0.01"/>
         </geometry>
     </visual>
     <inertial>
-      <mass value="0.01" />
+      <mass value="0.0001" />
+      <origin xyz="0 0 0" />
+      <inertia ixx="0.001" ixy="0.0" ixz="0.0"
+               iyy="0.001" iyz="0.0"
+               izz="0.001" />
+    </inertial>
+  </link> -->
+  <link name="dumper_bin">
+    <collision name='collision'>
+      <origin xyz="-0.3 0 0" rpy=" 0 0 1.57079"/>
+        <geometry>
+          <mesh filename="package://ssabot/meshes/meshes/dumper_bin.dae" scale="0.013 0.013 0.013"/>
+        </geometry>
+    </collision>
+    <visual name='dump_box_visual'>
+      <origin xyz=" -0.3 0 0.0" rpy="0 0 1.57079"/>
+        <geometry>
+          <mesh filename="package://ssabot/meshes/meshes/dumper_bin.dae" scale="0.013 0.013 0.013"/>
+        </geometry>
+    </visual>
+    <inertial>
+      <mass value="0.001" />
       <origin xyz="0 0 0" />
       <inertia ixx="0.001" ixy="0.0" ixz="0.0"
@@ -152,55 +162,3 @@
     </inertial>
   </link>
-<!-- add waffle_pi camera -->
-  <!-- <joint name="camera_joint" type="fixed">
-    <origin xyz="0.073 -0.011 0.084" rpy="0 0 0"/>
-    <parent link="base_link"/>
-    <child link="camera_link"/>
-  </joint>
-  <link name="camera_link">
-    <collision>
-      <origin xyz="0.005 0.011 0.013" rpy="0 0 0"/>
-      <geometry>
-        <box size="0.015 0.030 0.027"/>
-      </geometry>
-    </collision>
-  </link>
-  <joint name="camera_rgb_joint" type="fixed">
-    <origin xyz="0.003 0.011 0.009" rpy="0 0 0"/>
-    <parent link="camera_link"/>
-    <child link="camera_rgb_frame"/>
-  </joint>
-  <link name="camera_rgb_frame"/>
-  <joint name="camera_rgb_optical_joint" type="fixed">
-    <origin xyz="0 0 0" rpy="-1.57 0 -1.57"/>
-    <parent link="camera_rgb_frame"/>
-    <child link="camera_rgb_optical_frame"/>
-  </joint>
-  <link name="camera_rgb_optical_frame"/> -->
-  <!-- add second camera -->
-  <!-- <joint name="camera_joint2" type="fixed">
-    <origin xyz="0.073 -0.011 1.084" rpy="0 0 0"/>
-    <parent link="base_link"/>
-    <child link="camera_link2"/>
-  </joint>
-  <link name="camera_link2">
-    <collision>
-      <origin xyz="0.005 0.011 0.013" rpy="0 0 0"/>
-      <geometry>
-        <box size="0.015 0.030 0.027"/>
-      </geometry>
-    </collision>
-  </link>
-  <joint name="camera_rgb_joint2" type="fixed">
-    <origin xyz="0.003 0.011 0.009" rpy="0 0 0"/>
-    <parent link="camera_link2"/>
-    <child link="camera_rgb_frame2"/>
-  </joint>
-  <link name="camera_rgb_frame2"/>
-  <joint name="camera_rgb_optical_joint2" type="fixed">
-    <origin xyz="0 0 0" rpy="-1.57 0 -1.57"/>
-    <parent link="camera_rgb_frame2"/>
-    <child link="camera_rgb_optical_frame2"/>
-  </joint>
-  <link name="camera_rgb_optical_frame2"/> -->
 </robot>

File: ssapang_ws/src/ssabot/urdf/turtlebot3_waffle.urdf.xacro (robot description, xacro)
@@ -48,7 +48,7 @@
     </collision> -->
     <visual>
-      <origin xyz="-0.05 0 0.14" rpy="0 0 0"/>
-      <geometry>
-        <cylinder length="0.02" radius="0.005"/>
+	  <origin xyz="-0.05 0 0.14" rpy="0 0 0"/>
+      <geometry>
+        <cylinder length="0.03" radius="0.025"/>
       </geometry>
       <material name="red"/>
@@ -65,11 +65,11 @@
     <origin xyz="0 0 0" rpy="0 0 0"/>
     <axis xyz="0 0 1"/>
-    <limit effort="30" lower="-0.1" upper="0.3" velocity="0.171"/>
+    <limit effort="30" lower="-0.1" upper="0.015" velocity="0.171"/>
   </joint>
   <link name="piston_link2">
     <visual>
-      <origin xyz="-0.05 0 0.16" rpy="0 0 0"/>
-      <geometry>
-        <cylinder length="0.02" radius="0.01"/>
+	  <origin xyz="-0.05 0 0.16" rpy="0 0 0"/>
+      <geometry>
+        <cylinder length="0.02" radius="0.015"/>
       </geometry>
       <material name="orange"/>
@@ -87,14 +87,14 @@
   <link name="piston_plate">
     <visual>
-      <origin xyz="-0.064 0 0.17" rpy="0 0 1.57"/>
-      <geometry>
-        <mesh filename="package://ssabot/meshes/piston/untitled.dae" scale="0.005  0.005  0.01"/>
-      </geometry>
-      <material name="dark"/>
-    </visual>
-    <collision>
-      <origin xyz="-0.064 0 0.17" rpy="0 0 1.57"/>
-      <geometry>
-        <mesh filename="package://ssabot/meshes/piston/untitled.dae" scale="0.005  0.005 0.01"/>
+      <origin xyz="-0.05 0 0.16" rpy="0 0 1.57"/>
+      <geometry>
+        <mesh filename="package://ssabot/meshes/piston/untitled1.dae" scale="0.01  0.01  0.01"/>
+      </geometry>
+      <material name="dark"/>
+    </visual>
+    <collision>
+      <origin xyz="-0.05 0 0.16" rpy="0 0 1.57"/>
+      <geometry>
+        <mesh filename="package://ssabot/meshes/piston/untitled1.dae" scale="0.01  0.01 0.01"/>
       </geometry>
     </collision>

Commit message: [modified] ssapang map

File: ssapang_ws/src/ssabot/urdf/turtlebot3_burger.gazebo.xacro (robot description, xacro)
@@ -1,17 +1,20 @@
 <?xml version="1.0"?>
 <robot name="turtlebot3_burger_sim" xmlns:xacro="http://ros.org/wiki/xacro">
-  <xacro:arg name="laser_visual" default="false"/>
-  <xacro:arg name="imu_visual"   default="false"/>
-  <xacro:arg name="camera_visual" default="false"/>
+  <xacro:arg name="laser_visual" default="false" />
+  <xacro:arg name="imu_visual" default="false" />
+  <xacro:arg name="camera_visual" default="false" />
   <transmission name="dump_bin_actuator">
-          <type>transmission_interface/SimpleTransmission</type>
-          <joint name="dump_joint">
-              <hardwareInterface>hardware_interface/EffortJointInterface</hardwareInterface>
-          </joint>
-          <actuator name="dump_motor">
-              <hardwareInterface>hardware_interface/EffortJointInterface</hardwareInterface>
-              <mechanicalReduction>1</mechanicalReduction>
-          </actuator>
-    </transmission>
+    <type>transmission_interface/SimpleTransmission</type>
+    <joint name="dump_joint">
+      <hardwareInterface>hardware_interface/EffortJointInterface</hardwareInterface>
+    </joint>
+    <actuator name="dump_motor">
+      <hardwareInterface>hardware_interface/EffortJointInterface</hardwareInterface>
+      <mechanicalReduction>1</mechanicalReduction>
+    </actuator>
+  </transmission>
+  <gazebo reference="dumper_bin">
+    <material>Gazebo/Grass</material>
+  </gazebo>
   <gazebo>
     <plugin name="gazebo_ros_control" filename="libgazebo_ros_control.so">

File: ssapang_ws/src/ssabot/urdf/turtlebot3_burger.urdf.xacro (robot description, xacro)
@@ -148,5 +148,5 @@
         </geometry>
     </collision>
-    <visual name='dump_box_visual'>
+    <visual >
       <origin xyz=" -0.3 0 0.0" rpy="0 0 1.57079"/>
         <geometry>

File: ssapang_ws/src/ssabot/urdf/turtlebot3_waffle.urdf.xacro (robot description, xacro)
@@ -65,11 +65,11 @@
     <origin xyz="0 0 0" rpy="0 0 0"/>
     <axis xyz="0 0 1"/>
-    <limit effort="30" lower="-0.1" upper="0.015" velocity="0.171"/>
+    <limit effort="30" lower="-0.1" upper="0.02" velocity="0.171"/>
   </joint>
   <link name="piston_link2">
     <visual>
-	  <origin xyz="-0.05 0 0.16" rpy="0 0 0"/>
-      <geometry>
-        <cylinder length="0.02" radius="0.015"/>
+	  <origin xyz="-0.05 0 0.162" rpy="0 0 0"/>
+      <geometry>
+        <cylinder length="0.025" radius="0.015"/>
       </geometry>
       <material name="orange"/>

Commit message: [Add] shelf model

File: ssapang_ws/src/ssabot/urdf/turtlebot3_burger.gazebo.xacro (robot description, xacro)
@@ -4,4 +4,18 @@
   <xacro:arg name="imu_visual"   default="false"/>
   <xacro:arg name="camera_visual" default="false"/>
+  <transmission name="dump_bin_actuator">
+          <type>transmission_interface/SimpleTransmission</type>
+          <joint name="dump_joint">
+              <hardwareInterface>hardware_interface/EffortJointInterface</hardwareInterface>
+          </joint>
+          <actuator name="dump_motor">
+              <hardwareInterface>hardware_interface/EffortJointInterface</hardwareInterface>
+              <mechanicalReduction>1</mechanicalReduction>
+          </actuator>
+    </transmission>
+  <gazebo>
+    <plugin name="gazebo_ros_control" filename="libgazebo_ros_control.so">
+    </plugin>
+  </gazebo>
   <gazebo reference="base_link">
     <material>Gazebo/DarkGrey</material>

File: ssapang_ws/src/ssabot/urdf/turtlebot3_burger.urdf.xacro (robot description, xacro)
@@ -57,5 +57,5 @@
                iyy="2.1192413e-05" iyz="-2.4400107e-11"
                izz="4.0712558e-05" />
-      </inertial>
+    </inertial>
   </link>
   <joint name="wheel_right_joint" type="continuous">
@@ -113,25 +113,35 @@
   </joint>
   <link name="imu_link"/>
-  <joint name="scan_joint" type="fixed">
+  <joint name="dump_joint" type="revolute">
     <parent link="base_link"/>
-    <child link="base_scan"/>
-    <origin xyz="0 0 0.28" rpy="0 0 0"/>
+    <child link="dumper_bin"/>
+    <origin xyz="0.2 0 0.28" rpy="0 0 0"/>
+    <axis xyz="0 1 0"/>
+    <limit effort="1" velocity="1" lower="0" upper="0.6"/>
   </joint>
-  <link name="base_scan">
-    <!-- <visual>
-      <origin xyz="0 0 0.0" rpy="0 0 0"/>
-      <geometry>
-        <mesh filename="package://ssabot/meshes/sensors/lds.stl" scale="0.001 0.001 0.001"/>
-      </geometry>
-      <material name="dark"/>
+  <!-- <link name="dumper_bin">
+    <collision name='collision'>
+      <origin xyz="-0.15 0 0" rpy=" 0 0 1.57079"/>
+        <geometry>
+          <box size="0.3 0.3 0.01"/>
+        </geometry>
+    </collision>
+    <visual name='dump_box_visual'>
+      <origin xyz=" -0.15 0 0.0" rpy="0 0 1.57079"/>
+        <geometry>
+          <box size="0.3 0.3 0.01"/>
+        </geometry>
     </visual>
-    <collision>
-      <origin xyz="0.015 0 -0.0065" rpy="0 0 0"/>
-      <geometry>
-        <cylinder length="0.0315" radius="0.055"/>
-      </geometry>
-    </collision> -->
+    <inertial>
+      <mass value="0.0001" />
+      <origin xyz="0 0 0" />
+      <inertia ixx="0.001" ixy="0.0" ixz="0.0"
+               iyy="0.001" iyz="0.0"
+               izz="0.001" />
+    </inertial>
+  </link> -->
+  <link name="dumper_bin">
     <collision name='collision'>
-      <origin xyz="0 0 0" rpy=" 0 0 0"/>
+      <origin xyz="-0.3 0 0" rpy=" 0 0 1.57079"/>
         <geometry>
           <mesh filename="package://ssabot/meshes/meshes/dumper_bin.dae" scale="0.015 0.015 0.015"/>
@@ -139,5 +149,5 @@
     </collision>
     <visual name='dump_box_visual'>
-      <origin xyz=" 0 0 0.0" rpy="0 0 1.57079"/>
+      <origin xyz=" -0.3 0 0.0" rpy="0 0 1.57079"/>
         <geometry>
           <mesh filename="package://ssabot/meshes/meshes/dumper_bin.dae" scale="0.015 0.015 0.015"/>
@@ -145,5 +155,5 @@
     </visual>
     <inertial>
-      <mass value="0.01" />
+      <mass value="0.001" />
       <origin xyz="0 0 0" />
       <inertia ixx="0.001" ixy="0.0" ixz="0.0"
@@ -152,55 +162,3 @@
     </inertial>
   </link>
-<!-- add waffle_pi camera -->
-  <!-- <joint name="camera_joint" type="fixed">
-    <origin xyz="0.073 -0.011 0.084" rpy="0 0 0"/>
-    <parent link="base_link"/>
-    <child link="camera_link"/>
-  </joint>
-  <link name="camera_link">
-    <collision>
-      <origin xyz="0.005 0.011 0.013" rpy="0 0 0"/>
-      <geometry>
-        <box size="0.015 0.030 0.027"/>
-      </geometry>
-    </collision>
-  </link>
-  <joint name="camera_rgb_joint" type="fixed">
-    <origin xyz="0.003 0.011 0.009" rpy="0 0 0"/>
-    <parent link="camera_link"/>
-    <child link="camera_rgb_frame"/>
-  </joint>
-  <link name="camera_rgb_frame"/>
-  <joint name="camera_rgb_optical_joint" type="fixed">
-    <origin xyz="0 0 0" rpy="-1.57 0 -1.57"/>
-    <parent link="camera_rgb_frame"/>
-    <child link="camera_rgb_optical_frame"/>
-  </joint>
-  <link name="camera_rgb_optical_frame"/> -->
-  <!-- add second camera -->
-  <!-- <joint name="camera_joint2" type="fixed">
-    <origin xyz="0.073 -0.011 1.084" rpy="0 0 0"/>
-    <parent link="base_link"/>
-    <child link="camera_link2"/>
-  </joint>
-  <link name="camera_link2">
-    <collision>
-      <origin xyz="0.005 0.011 0.013" rpy="0 0 0"/>
-      <geometry>
-        <box size="0.015 0.030 0.027"/>
-      </geometry>
-    </collision>
-  </link>
-  <joint name="camera_rgb_joint2" type="fixed">
-    <origin xyz="0.003 0.011 0.009" rpy="0 0 0"/>
-    <parent link="camera_link2"/>
-    <child link="camera_rgb_frame2"/>
-  </joint>
-  <link name="camera_rgb_frame2"/>
-  <joint name="camera_rgb_optical_joint2" type="fixed">
-    <origin xyz="0 0 0" rpy="-1.57 0 -1.57"/>
-    <parent link="camera_rgb_frame2"/>
-    <child link="camera_rgb_optical_frame2"/>
-  </joint>
-  <link name="camera_rgb_optical_frame2"/> -->
 </robot>

File: ssapang_ws/src/ssabot/urdf/turtlebot3_waffle.gazebo.xacro (robot description, xacro)
@@ -76,5 +76,5 @@
       <wheelDiameter>0.066</wheelDiameter>
       <wheelAcceleration>1</wheelAcceleration>
-      <wheelTorque>10</wheelTorque>
+      <wheelTorque>20</wheelTorque>
       <rosDebugLevel>na</rosDebugLevel>
     </plugin>
@@ -141,8 +141,8 @@
   </gazebo>
   <gazebo reference="piston_plate">
-    <mu1>0.1</mu1>
-    <mu2>0.1</mu2>
+    <mu1>1</mu1>
+    <mu2>1</mu2>
     <kp>1000000.0</kp>
-    <kd>100.0</kd>
+    <kd>1000.0</kd>
     <material>Gazebo/FlatBlack</material>
   </gazebo>

File: ssapang_ws/src/ssabot/urdf/turtlebot3_waffle.urdf.xacro (robot description, xacro)
@@ -48,7 +48,7 @@
     </collision> -->
     <visual>
-	  <origin xyz="-0.05 0 0.14" rpy="0 0 0"/>
-      <geometry>
-        <cylinder length="0.02" radius="0.005"/>
+	  <origin xyz="-0.05 0 0.12" rpy="0 0 0"/>
+      <geometry>
+        <cylinder length="0.03" radius="0.025"/>
       </geometry>
       <material name="red"/>
@@ -65,11 +65,11 @@
     <origin xyz="0 0 0" rpy="0 0 0"/>
     <axis xyz="0 0 1"/>
-    <limit effort="30" lower="-0.1" upper="0.3" velocity="0.171"/>
+    <limit effort="30" lower="-0.1" upper="0.05" velocity="0.171"/>
   </joint>
   <link name="piston_link2">
     <visual>
-	  <origin xyz="-0.05 0 0.16" rpy="0 0 0"/>
-      <geometry>
-        <cylinder length="0.02" radius="0.01"/>
+	  <origin xyz="-0.05 0 0.08" rpy="0 0 0"/>
+      <geometry>
+        <cylinder length="0.08" radius="0.015"/>
       </geometry>
       <material name="orange"/>
@@ -87,14 +87,14 @@
   <link name="piston_plate">
     <visual>
-      <origin xyz="-0.05 0 0.17" rpy="0 0 1.57"/>
-      <geometry>
-        <mesh filename="package://ssabot/meshes/piston/piston_plate.dae" scale="0.015 0.015 0.015"/>
-      </geometry>
-      <material name="dark"/>
-    </visual>
-    <collision>
-      <origin xyz="-0.05 0 0.17" rpy="0 0 1.57"/>
-      <geometry>
-        <mesh filename="package://ssabot/meshes/piston/piston_plate.dae" scale="0.015 0.015 0.015"/>
+      <origin xyz="0 0 0.1" rpy="0 0 1.57"/>
+      <geometry>
+        <mesh filename="package://ssabot/meshes/piston/fix_plate.dae" scale="0.01  0.01  0.01"/>
+      </geometry>
+      <material name="dark"/>
+    </visual>
+    <collision>
+      <origin xyz="0 0 0.1" rpy="0 0 1.57"/>
+      <geometry>
+        <mesh filename="package://ssabot/meshes/piston/fix_plate.dae" scale="0.01  0.01 0.01"/>
       </geometry>
     </collision>
