Commit message: [Feat] Finally, i move itgit add .!

File: ssapang_ws/src/ssabot/urdf/push_robot.gazebo.xacro (robot description, xacro)
@@ -1,4 +1,14 @@
 <?xml version="1.0"?>
 <robot name="push_robot" xmlns:xacro="http://ros.org/wiki/xacro">
+    <transmission name="actuator1">
+        <type>transmission_interface/SimpleTransmission</type>
+        <joint name="virtual_joint1">
+            <hardwareInterface>hardware_interface/EffortJointInterface</hardwareInterface>
+        </joint>
+        <actuator name="push_motor1">
+            <hardwareInterface>hardware_interface/EffortJointInterface</hardwareInterface>
+            <mechanicalReduction>1</mechanicalReduction>
+        </actuator>
+    </transmission>
     <gazebo>
         <plugin name="joint_state_publisher" filename="libgazebo_ros_joint_state_publisher.so">
@@ -8,4 +18,5 @@
     <gazebo>
         <plugin name="gazebo_ros_control" filename="libgazebo_ros_control.so">
+            <robotNamespace>/push_robot</robotNamespace>
         </plugin>
     </gazebo>

File: ssapang_ws/src/ssabot/urdf/push_robot.urdf.xacro (robot description, xacro)
@@ -38,7 +38,7 @@
     <parent link="base_link"/>
     <child link="virtual_link1"/>
-    <origin xyz="0 0 0" rpy="0 0 0"/>
+    <origin xyz="0 0 1" rpy="0 0 0"/>
     <axis xyz="0 1 0"/>
-    <limit effort="30" lower="-0.3" upper="0.3" velocity="0.171"/>
+    <limit effort="5" lower="-1" upper="1" velocity="0.171"/>
   </joint>
   <link name="virtual_link1">
@@ -173,17 +173,14 @@
     </inertial>
   </link>
-  <transmission name="actuator1">
+  <!-- <transmission name="actuator1">
     <type>transmission_interface/SimpleTransmission</type>
     <joint name="virtual_joint1">
       <hardwareInterface>hardware_interface/EffortJointInterface</hardwareInterface>
     </joint>
-    <!-- <joint name="virtual_joint3">
-      <hardwareInterface>hardware_interface/EffortJointInterface</hardwareInterface>
-    </joint> -->
     <actuator name="push_motor1">
       <hardwareInterface>hardware_interface/EffortJointInterface</hardwareInterface>
       <mechanicalReduction>1</mechanicalReduction>
     </actuator>
-  </transmission>
+  </transmission> -->
   <!--  -->
   <!-- <link name="piston_link2">

Commit message: [Add] push_robot 구현

File: ssapang_ws/src/ssabot/urdf/push_robot.gazebo.xacro (robot description, xacro)
@@ -1,7 +1,27 @@
 <?xml version="1.0"?>
 <robot name="push_robot" xmlns:xacro="http://ros.org/wiki/xacro">
-    <transmission name="actuator1">
+    <transmission name="virtual_actuator1">
         <type>transmission_interface/SimpleTransmission</type>
         <joint name="virtual_joint1">
+            <hardwareInterface>hardware_interface/EffortJointInterface</hardwareInterface>
+        </joint>
+        <actuator name="virtual_motor1">
+            <hardwareInterface>hardware_interface/EffortJointInterface</hardwareInterface>
+            <mechanicalReduction>1</mechanicalReduction>
+        </actuator>
+    </transmission>
+    <transmission name="virtual_actuator2">
+        <type>transmission_interface/SimpleTransmission</type>
+        <joint name="virtual_joint2">
+            <hardwareInterface>hardware_interface/EffortJointInterface</hardwareInterface>
+        </joint>
+        <actuator name="virtual_motor2">
+            <hardwareInterface>hardware_interface/EffortJointInterface</hardwareInterface>
+            <mechanicalReduction>1</mechanicalReduction>
+        </actuator>
+    </transmission>
+    <transmission name="push_actuator1">
+        <type>transmission_interface/SimpleTransmission</type>
+        <joint name="push_joint1">
             <hardwareInterface>hardware_interface/EffortJointInterface</hardwareInterface>
         </joint>
@@ -11,4 +31,15 @@
         </actuator>
     </transmission>
+    <transmission name="push_actuator2">
+        <type>transmission_interface/SimpleTransmission</type>
+        <joint name="push_joint2">
+            <hardwareInterface>hardware_interface/EffortJointInterface</hardwareInterface>
+        </joint>
+        <actuator name="push_motor2">
+            <hardwareInterface>hardware_interface/EffortJointInterface</hardwareInterface>
+            <mechanicalReduction>1</mechanicalReduction>
+        </actuator>
+    </transmission>
+<!--
     <gazebo>
         <plugin name="joint_state_publisher" filename="libgazebo_ros_joint_state_publisher.so">
@@ -16,4 +47,5 @@
         </plugin>
     </gazebo>
+     -->
     <gazebo>
         <plugin name="gazebo_ros_control" filename="libgazebo_ros_control.so">
@@ -21,5 +53,5 @@
         </plugin>
     </gazebo>
-    <gazebo reference="base_link">
+    <gazebo reference="base_link1">
         <material>Gazebo/Black</material>
     </gazebo>

File: ssapang_ws/src/ssabot/urdf/push_robot.urdf.xacro (robot description, xacro)
@@ -9,40 +9,66 @@
   <joint name="base_joint" type="fixed">
     <parent link="base_footprint"/>
-    <child link="base_link" />
+    <child link="base_link1" />
+    <origin xyz="0 0 0" rpy="0 0 0"/>
+  </joint>
+  <link name="base_link1">
+    <visual>
+      <origin xyz="0 0 0.05" rpy="0 0 0"/>
+      <geometry>
+        <!-- <box size="0.1 0.1 0.1"/> -->
+        <box size="0.5 1 0.01"/>
+      </geometry>
+    </visual>
+    <collision>
+      <origin xyz="0 0 0.05" rpy="0 0 0"/>
+      <geometry>
+        <!-- <box size="0.1 0.1 0.1"/> -->
+        <box size="0.5 1 0.01"/>
+      </geometry>
+    </collision>
+    <inertial>
+      <origin xyz="0 0 0" rpy="0 0 0"/>
+      <mass value="1.3729096e+01"/>
+      <inertia ixx="8.7002718e-03" ixy="-4.7576583e-05" ixz="1.1160499e-04"
+               iyy="8.6195418e-03" iyz="-3.5422299e-06"
+               izz="1.4612727e-02" />
+    </inertial>
+  </link>
+   <joint name="virtual_joint1" type="prismatic">
+    <parent link="base_link1"/>
+    <child link="base_link2"/>
+    <origin xyz="0 0 0.05" rpy="0 0 0"/>
+    <axis xyz="0 1 0"/>
+    <limit effort="5" lower="-0.5" upper="0.5" velocity="0.171"/>
+  </joint>
+  <link name="base_link2">
+    <visual>
+      <origin xyz="0 0 0.05" rpy="0 0 0"/>
+      <geometry>
+        <box size="0.1 0.1 0.1"/>
+      </geometry>
+    </visual>
+    <!-- <collision>
+      <origin xyz="0 0 0.3" rpy="0 0 0"/>
+      <geometry>
+          <box size="0.1 0.1 0.1"/>
+      </geometry>
+    </collision> -->
+    <inertial>
+      <origin xyz="0 0 0" rpy="0 0 0"/>
+      <mass value="1.3729096e-05"/>
+      <inertia ixx="8.7002718e-03" ixy="-4.7576583e-05" ixz="1.1160499e-04"
+               iyy="8.6195418e-03" iyz="-3.5422299e-06"
+               izz="1.4612727e-02" />
+    </inertial>
+  </link>
+  <joint name="fixed_joint" type="fixed">
+    <parent link="base_link2"/>
+    <child link="virtual_link1"/>
     <origin xyz="0 0 0.5" rpy="0 0 0"/>
   </joint>
-  <link name="base_link">
-    <visual>
-      <origin xyz="0 0 0.05" rpy="0 0 0"/>
-      <geometry>
-        <!-- <box size="0.1 0.1 0.1"/> -->
-        <box size="0.5 0.5 0.01"/>
-      </geometry>
-    </visual>
-    <collision>
-      <origin xyz="0 0 0.05" rpy="0 0 0"/>
-      <geometry>
-        <!-- <box size="0.1 0.1 0.1"/> -->
-        <box size="0.5 0.5 0.01"/>
-      </geometry>
-    </collision>
-    <inertial>
-      <origin xyz="0 0 0" rpy="0 0 0"/>
-      <mass value="1.3729096e+00"/>
-      <inertia ixx="8.7002718e-03" ixy="-4.7576583e-05" ixz="1.1160499e-04"
-               iyy="8.6195418e-03" iyz="-3.5422299e-06"
-               izz="1.4612727e-02" />
-    </inertial>
-  </link>
-  <joint name="virtual_joint1" type="prismatic">
-    <parent link="base_link"/>
-    <child link="virtual_link1"/>
-    <origin xyz="0 0 1" rpy="0 0 0"/>
-    <axis xyz="0 1 0"/>
-    <limit effort="5" lower="-1" upper="1" velocity="0.171"/>
-  </joint>
   <link name="virtual_link1">
     <visual>
-      <origin xyz="0 0 0.5" rpy="0 0 0"/>
+      <origin xyz="0 0 0" rpy="0 0 0"/>
       <geometry>
         <cylinder length="1" radius="0.01"/>
@@ -57,5 +83,5 @@
     <inertial>
       <origin xyz="0 0 0" rpy="0 0 0"/>
-      <mass value="1.3729096e+00"/>
+      <mass value="1.3729096e-05"/>
       <inertia ixx="8.7002718e-03" ixy="-4.7576583e-05" ixz="1.1160499e-04"
                iyy="8.6195418e-03" iyz="-3.5422299e-06"
@@ -64,63 +90,37 @@
   </link>
   <joint name="virtual_joint2" type="prismatic">
+    <parent link="base_link1"/>
+    <child link="virtual_link2"/>
+    <origin xyz="0 0 0.55" rpy="0 0 0"/>
+    <axis xyz="0 0 1"/>
+    <limit effort="5" lower="-0.5" upper="0.5" velocity="0.171"/>
+  </joint>
+  <link name="virtual_link2">
+    <visual>
+      <origin xyz="0 0 0" rpy="-1.57 0 0"/>
+      <geometry>
+        <cylinder length="1" radius="0.01"/>
+      </geometry>
+    </visual>
+    <!-- <collision>
+      <origin xyz="0 0.1 0" rpy="0 0 0"/>
+      <geometry>
+          <box size="0.1 0.1 0.1"/>
+      </geometry>
+    </collision> -->
+    <inertial>
+      <origin xyz="0 0 0" rpy="-1.57 0 0"/>
+      <mass value="1.3729096e-05"/>
+      <inertia ixx="8.7002718e-03" ixy="-4.7576583e-05" ixz="1.1160499e-04"
+               iyy="8.6195418e-03" iyz="-3.5422299e-06"
+               izz="1.4612727e-02" />
+    </inertial>
+  </link>
+  <joint name="push_joint1" type="prismatic">
     <parent link="virtual_link1"/>
-    <child link="virtual_link2"/>
+    <child link="push_link1"/>
     <origin xyz="0 0 0" rpy="0 0 0"/>
     <axis xyz="0 0 1"/>
-    <limit effort="30" lower="-0.001" upper="0.001" velocity="0.171"/>
-  </joint>
-  <link name="virtual_link2">
-    <visual>
-      <origin xyz="0 0 0" rpy="-1.57 0 0"/>
-      <geometry>
-        <cylinder length="1" radius="0.01"/>
-      </geometry>
-    </visual>
-    <!-- <collision>
-      <origin xyz="0 0.1 0" rpy="0 0 0"/>
-      <geometry>
-          <box size="0.1 0.1 0.1"/>
-      </geometry>
-    </collision> -->
-    <inertial>
-      <origin xyz="0 0 0" rpy="0 0 0"/>
-      <mass value="1.3729096e+00"/>
-      <inertia ixx="8.7002718e-03" ixy="-4.7576583e-05" ixz="1.1160499e-04"
-               iyy="8.6195418e-03" iyz="-3.5422299e-06"
-               izz="1.4612727e-02" />
-    </inertial>
-  </link>
-  <joint name="virtual_joint3" type="prismatic">
-    <parent link="virtual_link2"/>
-    <child link="virtual_link3"/>
-    <origin xyz="0 0 0" rpy="0 0 0"/>
-    <axis xyz="0 1 0"/>
-    <limit effort="30" lower="-0.001" upper="0.001" velocity="0.171"/>
-  </joint>
-  <link name="virtual_link3">
-    <visual>
-      <origin xyz="0 0 0" rpy="0 0 0"/>
-      <geometry>
-        <box size="0.1 0.1 0.1"/>
-      </geometry>
-    </visual>
-    <!-- <collision>
-      <origin xyz="0 0 0.05" rpy="0 0 0"/>
-      <geometry>
-          <box size="0.1 0.1 0.1"/>
-      </geometry>
-    </collision> -->
-    <inertial>
-      <origin xyz="0 0 0" rpy="0 0 0"/>
-      <mass value="1.3729096e+00"/>
-      <inertia ixx="8.7002718e-03" ixy="-4.7576583e-05" ixz="1.1160499e-04"
-               iyy="8.6195418e-03" iyz="-3.5422299e-06"
-               izz="1.4612727e-02" />
-    </inertial>
-  </link>
-  <joint name="push_joint1" type="fixed">
-    <parent link="virtual_link3"/>
-    <child link="push_link1"/>
-    <origin xyz="0 0 0" rpy="0 0 0"/>
+    <limit effort="5" lower="-0.5" upper="0.5" velocity="0.171"/>
   </joint>
   <link name="push_link1">
@@ -139,5 +139,5 @@
     <inertial>
       <origin xyz="0 0 0" rpy="0 0 0"/>
-      <mass value="1.3729096e+00"/>
+      <mass value="1.3729096e-05"/>
       <inertia ixx="8.7002718e-03" ixy="-4.7576583e-05" ixz="1.1160499e-04"
                iyy="8.6195418e-03" iyz="-3.5422299e-06"
@@ -150,5 +150,5 @@
     <origin xyz="0 0 0" rpy="0 0 0"/>
     <axis xyz="1 0 0"/>
-    <limit effort="30" lower="-0.001" upper="0.001" velocity="0.171"/>
+    <limit effort="30" lower="-0.1" upper="0.1" velocity="0.171"/>
   </joint>
   <link name="push_link2">
@@ -167,5 +167,5 @@
     <inertial>
       <origin xyz="0 0 0" rpy="0 0 0"/>
-      <mass value="1.3729096e+00"/>
+      <mass value="1.3729096e-05"/>
       <inertia ixx="8.7002718e-03" ixy="-4.7576583e-05" ixz="1.1160499e-04"
                iyy="8.6195418e-03" iyz="-3.5422299e-06"

Commit message: [Add] Spawn multiple push_robots

File: ssapang_ws/src/ssabot/urdf/push_robot.gazebo.xacro (robot description, xacro)
@@ -50,5 +50,4 @@
     <gazebo>
         <plugin name="gazebo_ros_control" filename="libgazebo_ros_control.so">
-            <robotNamespace>/push_robot</robotNamespace>
         </plugin>
     </gazebo>

File: ssapang_ws/src/ssabot/urdf/push_robot.urdf.xacro (robot description, xacro)
@@ -123,5 +123,5 @@
     <origin xyz="0 0 0" rpy="0 0 0"/>
     <axis xyz="1 0 0"/>
-    <limit effort="0.001" lower="-0.1" upper="0.1" velocity="0.0001"/>
+    <limit effort="50" lower="-0.3" upper="0.3" velocity="0.001"/>
   </joint>
   <link name="push_link2">

Commit message: [Add] push and catch

File: ssapang_ws/src/ssabot/urdf/push_robot.gazebo.xacro (robot description, xacro)
@@ -52,7 +52,4 @@
         </plugin>
     </gazebo>
-    <gazebo reference="base_link1">
-        <material>Gazebo/Black</material>
-    </gazebo>
     <gazebo reference="virtual_link1">
         <material>Gazebo/Orange</material>

File: ssapang_ws/src/ssabot/urdf/push_robot.urdf.xacro (robot description, xacro)
@@ -39,5 +39,5 @@
     <origin xyz="0 0 1" rpy="0 0 0"/>
     <axis xyz="0 1 0"/>
-    <limit effort="0.03" lower="-0.5" upper="0.5" velocity="0.0001"/>
+    <limit effort="0.03" lower="-0.8" upper="0.8" velocity="0.0001"/>
   </joint>
   <link name="virtual_link1">
@@ -67,5 +67,5 @@
     <origin xyz="0 0 1" rpy="0 0 0"/>
     <axis xyz="0 0 1"/>
-    <limit effort="0.03" lower="-0.5" upper="0.5" velocity="0.0001"/>
+    <limit effort="0.03" lower="-0.8" upper="0.8" velocity="0.0001"/>
   </joint>
   <link name="virtual_link2">

File: ssapang_ws/src/ssabot/urdf/turtlebot3_burger.gazebo.xacro (robot description, xacro)
@@ -17,4 +17,7 @@
     <plugin name="gazebo_ros_control" filename="libgazebo_ros_control.so">
     </plugin>
+  </gazebo>
+  <gazebo reference="dumper_bin">
+    <material>Gazebo/Gold</material>
   </gazebo>
   <gazebo reference="base_link">

File: ssapang_ws/src/ssabot/urdf/turtlebot3_burger.urdf.xacro (robot description, xacro)
@@ -1,5 +1,5 @@
 <?xml version="1.0" ?>
 <robot name="turtlebot3_burger" xmlns:xacro="http://ros.org/wiki/xacro">
-  <xacro:include filename="$(find ssabot)/urdf/common_properties.xacro"/>
+  <!-- <xacro:include filename="$(find ssabot)/urdf/common_properties.xacro"/> -->
   <xacro:include filename="$(find ssabot)/urdf/turtlebot3_burger.gazebo.xacro"/>
   <link name="base_footprint"/>
@@ -15,5 +15,6 @@
         <mesh filename="package://ssabot/meshes/bases/burger_base.stl" scale="0.002 0.002 0.002"/>
       </geometry>
-      <material name="light_black"/>
+      <!-- <material name="light_black"/> -->
+      <material name="blue"/>
     </visual>
     <collision>
@@ -43,5 +44,5 @@
         <mesh filename="package://ssabot/meshes/wheels/left_tire.stl" scale="0.002 0.002 0.002"/>
       </geometry>
-      <material name="dark"/>
+      <!-- <material name="dark"/> -->
     </visual>
     <collision>
@@ -71,5 +72,5 @@
         <mesh filename="package://ssabot/meshes/wheels/right_tire.stl" scale="0.002 0.002 0.002"/>
       </geometry>
-      <material name="dark"/>
+      <!-- <material name="dark"/> -->
     </visual>
     <collision>
@@ -145,12 +146,12 @@
       <origin xyz="-0.3 0 0" rpy=" 0 0 1.57079"/>
         <geometry>
-          <mesh filename="package://ssabot/meshes/meshes/dumper_bin.dae" scale="0.015 0.015 0.015"/>
+          <mesh filename="package://ssabot/meshes/meshes/dumper_bin.dae" scale="0.013 0.013 0.013"/>
         </geometry>
     </collision>
-    <visual name='dump_box_visual'>
+    <visual>
       <origin xyz=" -0.3 0 0.0" rpy="0 0 1.57079"/>
-        <geometry>
-          <mesh filename="package://ssabot/meshes/meshes/dumper_bin.dae" scale="0.015 0.015 0.015"/>
-        </geometry>
+      <geometry>
+        <mesh filename="package://ssabot/meshes/meshes/dumper_bin.dae" scale="0.013 0.013 0.013"/>
+      </geometry>
     </visual>
     <inertial>
