Commit message: [del] ssapang

File: ssapang_ws/src/ssabot/urdf/push_robot.gazebo.xacro (robot description, xacro)
@@ -52,4 +52,10 @@
         </plugin>
     </gazebo>
+<<<<<<< HEAD
+=======
+    <gazebo reference="base_link1">
+        <material>Gazebo/Black</material>
+    </gazebo>
+>>>>>>> d2d46bd033c6114a82d2ed123778a13e47a874d7
     <gazebo reference="virtual_link1">
         <material>Gazebo/Orange</material>

File: ssapang_ws/src/ssabot/urdf/push_robot.urdf.xacro (robot description, xacro)
@@ -39,5 +39,9 @@
     <origin xyz="0 0 1" rpy="0 0 0"/>
     <axis xyz="0 1 0"/>
+<<<<<<< HEAD
     <limit effort="0.03" lower="-0.8" upper="0.8" velocity="0.0001"/>
+=======
+    <limit effort="0.03" lower="-0.5" upper="0.5" velocity="0.0001"/>
+>>>>>>> d2d46bd033c6114a82d2ed123778a13e47a874d7
   </joint>
   <link name="virtual_link1">
@@ -67,5 +71,9 @@
     <origin xyz="0 0 1" rpy="0 0 0"/>
     <axis xyz="0 0 1"/>
+<<<<<<< HEAD
     <limit effort="0.03" lower="-0.8" upper="0.8" velocity="0.0001"/>
+=======
+    <limit effort="0.03" lower="-0.5" upper="0.5" velocity="0.0001"/>
+>>>>>>> d2d46bd033c6114a82d2ed123778a13e47a874d7
   </joint>
   <link name="virtual_link2">

File: ssapang_ws/src/ssabot/urdf/turtlebot3_burger.gazebo.xacro (robot description, xacro)
@@ -1,7 +1,24 @@
 <?xml version="1.0"?>
 <robot name="turtlebot3_burger_sim" xmlns:xacro="http://ros.org/wiki/xacro">
-  <xacro:arg name="laser_visual" default="false"/>
-  <xacro:arg name="imu_visual"   default="false"/>
-  <xacro:arg name="camera_visual" default="false"/>
+  <xacro:arg name="laser_visual" default="false" />
+  <xacro:arg name="imu_visual" default="false" />
+  <xacro:arg name="camera_visual" default="false" />
+  <transmission name="dump_bin_actuator">
+    <type>transmission_interface/SimpleTransmission</type>
+    <joint name="dump_joint">
+      <hardwareInterface>hardware_interface/EffortJointInterface</hardwareInterface>
+    </joint>
+    <actuator name="dump_motor">
+      <hardwareInterface>hardware_interface/EffortJointInterface</hardwareInterface>
+      <mechanicalReduction>1</mechanicalReduction>
+    </actuator>
+  </transmission>
+  <gazebo reference="dumper_bin">
+    <material>Gazebo/Grass</material>
+  </gazebo>
+  <gazebo>
+    <plugin name="gazebo_ros_control" filename="libgazebo_ros_control.so">
+    </plugin>
+  </gazebo>
   <transmission name="dump_bin_actuator">
           <type>transmission_interface/SimpleTransmission</type>
@@ -142,4 +159,7 @@
     </sensor>
   </gazebo>
+<<<<<<< HEAD
+=======
+>>>>>>> d2d46bd033c6114a82d2ed123778a13e47a874d7
   <!-- dump_box -->
   <gazebo reference="dump_box_visual">
@@ -212,3 +232,6 @@
     </sensor>
   </gazebo> -->
+<<<<<<< HEAD
+=======
+>>>>>>> d2d46bd033c6114a82d2ed123778a13e47a874d7
 </robot>

File: ssapang_ws/src/ssabot/urdf/turtlebot3_burger.urdf.xacro (robot description, xacro)
@@ -142,5 +142,9 @@
     </inertial>
   </link> -->
+<<<<<<< HEAD
   <link name="dumper_bin">
+=======
+  <link name="dumper_bin">
+>>>>>>> d2d46bd033c6114a82d2ed123778a13e47a874d7
     <collision name='collision'>
       <origin xyz="-0.3 0 0" rpy=" 0 0 1.57079"/>
@@ -149,4 +153,5 @@
         </geometry>
     </collision>
+<<<<<<< HEAD
     <visual>
       <origin xyz=" -0.3 0 0.0" rpy="0 0 1.57079"/>
@@ -154,4 +159,11 @@
         <mesh filename="package://ssabot/meshes/meshes/dumper_bin.dae" scale="0.013 0.013 0.013"/>
       </geometry>
+=======
+    <visual >
+      <origin xyz=" -0.3 0 0.0" rpy="0 0 1.57079"/>
+        <geometry>
+          <mesh filename="package://ssabot/meshes/meshes/dumper_bin.dae" scale="0.013 0.013 0.013"/>
+        </geometry>
+>>>>>>> d2d46bd033c6114a82d2ed123778a13e47a874d7
     </visual>
     <inertial>

File: ssapang_ws/src/ssabot/urdf/turtlebot3_waffle.gazebo.xacro (robot description, xacro)
@@ -76,5 +76,5 @@
       <wheelDiameter>0.066</wheelDiameter>
       <wheelAcceleration>1</wheelAcceleration>
-      <wheelTorque>10</wheelTorque>
+      <wheelTorque>20</wheelTorque>
       <rosDebugLevel>na</rosDebugLevel>
     </plugin>
@@ -140,46 +140,10 @@
     </sensor>
   </gazebo>
-  <gazebo reference="camera_rgb_frame">
-    <sensor type="depth" name="realsense_R200">
-      <always_on>true</always_on>
-      <visualize>$(arg camera_visual)</visualize>
-      <camera>
-          <horizontal_fov>1.3439</horizontal_fov>
-          <image>
-              <width>1920</width>
-              <height>1080</height>
-              <format>R8G8B8</format>
-          </image>
-          <depth_camera></depth_camera>
-          <clip>
-              <near>0.03</near>
-              <far>100</far>
-          </clip>
-      </camera>
-      <plugin name="camera_controller" filename="libgazebo_ros_openni_kinect.so">
-        <baseline>0.2</baseline>
-        <alwaysOn>true</alwaysOn>
-        <updateRate>30.0</updateRate>
-        <cameraName>camera</cameraName>
-        <frameName>camera_rgb_optical_frame</frameName>
-        <imageTopicName>rgb/image_raw</imageTopicName>
-        <depthImageTopicName>depth/image_raw</depthImageTopicName>
-        <pointCloudTopicName>depth/points</pointCloudTopicName>
-        <cameraInfoTopicName>rgb/camera_info</cameraInfoTopicName>
-        <depthImageCameraInfoTopicName>depth/camera_info</depthImageCameraInfoTopicName>
-        <pointCloudCutoff>0.4</pointCloudCutoff>
-            <hackBaseline>0.07</hackBaseline>
-            <distortionK1>0.0</distortionK1>
-            <distortionK2>0.0</distortionK2>
-            <distortionK3>0.0</distortionK3>
-            <distortionT1>0.0</distortionT1>
-            <distortionT2>0.0</distortionT2>
-        <CxPrime>0.0</CxPrime>
-        <Cx>0.0</Cx>
-        <Cy>0.0</Cy>
-        <focalLength>0</focalLength>
-        <hackBaseline>0</hackBaseline>
-      </plugin>
-    </sensor>
+  <gazebo reference="piston_plate">
+    <mu1>1</mu1>
+    <mu2>1</mu2>
+    <kp>1000000.0</kp>
+    <kd>10000.0</kd>
+    <material>Gazebo/FlatBlack</material>
   </gazebo>
 </robot>

File: ssapang_ws/src/ssabot/urdf/turtlebot3_waffle.urdf.xacro (robot description, xacro)
@@ -50,5 +50,5 @@
 	  <origin xyz="-0.05 0 0.14" rpy="0 0 0"/>
       <geometry>
-        <cylinder length="0.02" radius="0.005"/>
+        <cylinder length="0.03" radius="0.025"/>
       </geometry>
       <material name="red"/>
@@ -65,11 +65,11 @@
     <origin xyz="0 0 0" rpy="0 0 0"/>
     <axis xyz="0 0 1"/>
-    <limit effort="30" lower="-0.1" upper="0.1" velocity="0.171"/>
+    <limit effort="30" lower="-0.1" upper="0.02" velocity="0.171"/>
   </joint>
   <link name="piston_link2">
     <visual>
-	  <origin xyz="-0.05 0 0.16" rpy="0 0 0"/>
-      <geometry>
-        <cylinder length="0.02" radius="0.01"/>
+	  <origin xyz="-0.05 0 0.162" rpy="0 0 0"/>
+      <geometry>
+        <cylinder length="0.025" radius="0.015"/>
       </geometry>
       <material name="orange"/>
@@ -87,17 +87,16 @@
   <link name="piston_plate">
     <visual>
-      <origin xyz="-0.05 0 0.17" rpy="0 0 1.57"/>
-      <geometry>
-        <mesh filename="package://ssabot/meshes/piston/piston_plate.dae" scale="0.015 0.015 0.015"/>
-      </geometry>
-      <material name="dark"/>
-    </visual>
-    <collision>
-      <origin xyz="-0.05 0 0.17" rpy="0 0 1.57"/>
-      <geometry>
-        <mesh filename="package://ssabot/meshes/piston/piston_plate.dae" scale="0.015 0.015 0.015"/>
-      </geometry>
-    </collision>
-<!--
+      <origin xyz="-0.05 0 0.16" rpy="0 0 1.57"/>
+      <geometry>
+        <mesh filename="package://ssabot/meshes/piston/untitled1.dae" scale="0.01  0.01  0.01"/>
+      </geometry>
+      <material name="dark"/>
+    </visual>
+    <collision>
+      <origin xyz="-0.05 0 0.16" rpy="0 0 1.57"/>
+      <geometry>
+        <mesh filename="package://ssabot/meshes/piston/untitled1.dae" scale="0.01  0.01 0.01"/>
+      </geometry>
+    </collision>
     <inertial>
       <mass value="0.114" />
@@ -106,5 +105,5 @@
                iyy="0.001" iyz="0.0"
                izz="0.001" />
-    </inertial> -->
+    </inertial>
   </link>
   <transmission name="waffle_tran">
@@ -248,54 +247,3 @@
     </inertial>
   </link>
-  <joint name="camera_joint" type="fixed">
-    <origin xyz="0.064 -0.065 0.094" rpy="0 0 0"/>
-    <parent link="base_link"/>
-    <child link="camera_link"/>
-  </joint>
-  <link name="camera_link">
-    <visual>
-     <origin xyz="0 0 0" rpy="1.57 0 1.57"/>
-      <geometry>
-       <mesh filename="package://ssabot/meshes/sensors/r200.dae" />
-      </geometry>
-    </visual>
-    <collision>
-      <origin xyz="0.003 0.065 0.007" rpy="0 0 0"/>
-      <geometry>
-        <box size="0.012 0.132 0.020"/>
-      </geometry>
-    </collision>
-    <!-- This inertial field needs doesn't contain reliable data!! -->
-<!--   <inertial>
-      <mass value="0.564" />
-      <origin xyz="0 0 0" />
-      <inertia ixx="0.003881243" ixy="0.0" ixz="0.0"
-               iyy="0.000498940" iyz="0.0"
-               izz="0.003879257" />
-    </inertial>-->
-  </link>
-  <joint name="camera_rgb_joint" type="fixed">
-    <origin xyz="${r200_cam_rgb_px} ${r200_cam_rgb_py} ${r200_cam_rgb_pz}" rpy="0 0 0"/>
-    <parent link="camera_link"/>
-    <child link="camera_rgb_frame"/>
-  </joint>
-  <link name="camera_rgb_frame"/>
-  <joint name="camera_rgb_optical_joint" type="fixed">
-    <origin xyz="0 0 0" rpy="-1.57 0 -1.57"/>
-    <parent link="camera_rgb_frame"/>
-    <child link="camera_rgb_optical_frame"/>
-  </joint>
-  <link name="camera_rgb_optical_frame"/>
-  <joint name="camera_depth_joint" type="fixed">
-    <origin xyz="${r200_cam_rgb_px} ${r200_cam_rgb_py + r200_cam_depth_offset} ${r200_cam_rgb_pz}" rpy="0 0 0"/>
-    <parent link="camera_link"/>
-    <child link="camera_depth_frame"/>
-  </joint>
-  <link name="camera_depth_frame"/>
-  <joint name="camera_depth_optical_joint" type="fixed">
-    <origin xyz="0 0 0" rpy="-1.57 0 -1.57"/>
-    <parent link="camera_depth_frame"/>
-    <child link="camera_depth_optical_frame"/>
-  </joint>
-  <link name="camera_depth_optical_frame"/>
 </robot>

Commit message: [Modify]

File: ssapang_ws/src/ssabot/urdf/push_robot.gazebo.xacro (robot description, xacro)
@@ -52,10 +52,4 @@
         </plugin>
     </gazebo>
-<<<<<<< HEAD
-=======
-    <gazebo reference="base_link1">
-        <material>Gazebo/Black</material>
-    </gazebo>
->>>>>>> d2d46bd033c6114a82d2ed123778a13e47a874d7
     <gazebo reference="virtual_link1">
         <material>Gazebo/Orange</material>

File: ssapang_ws/src/ssabot/urdf/push_robot.urdf.xacro (robot description, xacro)
@@ -39,9 +39,5 @@
     <origin xyz="0 0 1" rpy="0 0 0"/>
     <axis xyz="0 1 0"/>
-<<<<<<< HEAD
     <limit effort="0.03" lower="-0.8" upper="0.8" velocity="0.0001"/>
-=======
-    <limit effort="0.03" lower="-0.5" upper="0.5" velocity="0.0001"/>
->>>>>>> d2d46bd033c6114a82d2ed123778a13e47a874d7
   </joint>
   <link name="virtual_link1">
@@ -71,9 +67,5 @@
     <origin xyz="0 0 1" rpy="0 0 0"/>
     <axis xyz="0 0 1"/>
-<<<<<<< HEAD
     <limit effort="0.03" lower="-0.8" upper="0.8" velocity="0.0001"/>
-=======
-    <limit effort="0.03" lower="-0.5" upper="0.5" velocity="0.0001"/>
->>>>>>> d2d46bd033c6114a82d2ed123778a13e47a874d7
   </joint>
   <link name="virtual_link2">
@@ -125,5 +117,5 @@
     <origin xyz="0 0 0" rpy="0 0 0"/>
     <axis xyz="1 0 0"/>
-    <limit effort="60" lower="-1" upper="1" velocity="0.01"/>
+    <limit effort="0.185" lower="-1" upper="1" velocity="0.001"/>
   </joint>
   <link name="push_link2">

File: ssapang_ws/src/ssabot/urdf/turtlebot3_burger.gazebo.xacro (robot description, xacro)
@@ -1,24 +1,7 @@
 <?xml version="1.0"?>
 <robot name="turtlebot3_burger_sim" xmlns:xacro="http://ros.org/wiki/xacro">
-  <xacro:arg name="laser_visual" default="false" />
-  <xacro:arg name="imu_visual" default="false" />
-  <xacro:arg name="camera_visual" default="false" />
-  <transmission name="dump_bin_actuator">
-    <type>transmission_interface/SimpleTransmission</type>
-    <joint name="dump_joint">
-      <hardwareInterface>hardware_interface/EffortJointInterface</hardwareInterface>
-    </joint>
-    <actuator name="dump_motor">
-      <hardwareInterface>hardware_interface/EffortJointInterface</hardwareInterface>
-      <mechanicalReduction>1</mechanicalReduction>
-    </actuator>
-  </transmission>
-  <gazebo reference="dumper_bin">
-    <material>Gazebo/Grass</material>
-  </gazebo>
-  <gazebo>
-    <plugin name="gazebo_ros_control" filename="libgazebo_ros_control.so">
-    </plugin>
-  </gazebo>
+  <xacro:arg name="laser_visual" default="false"/>
+  <xacro:arg name="imu_visual"   default="false"/>
+  <xacro:arg name="camera_visual" default="false"/>
   <transmission name="dump_bin_actuator">
           <type>transmission_interface/SimpleTransmission</type>
@@ -159,7 +142,4 @@
     </sensor>
   </gazebo>
-<<<<<<< HEAD
-=======
->>>>>>> d2d46bd033c6114a82d2ed123778a13e47a874d7
   <!-- dump_box -->
   <gazebo reference="dump_box_visual">
@@ -232,6 +212,3 @@
     </sensor>
   </gazebo> -->
-<<<<<<< HEAD
-=======
->>>>>>> d2d46bd033c6114a82d2ed123778a13e47a874d7
 </robot>

File: ssapang_ws/src/ssabot/urdf/turtlebot3_burger.urdf.xacro (robot description, xacro)
@@ -142,9 +142,5 @@
     </inertial>
   </link> -->
-<<<<<<< HEAD
   <link name="dumper_bin">
-=======
-  <link name="dumper_bin">
->>>>>>> d2d46bd033c6114a82d2ed123778a13e47a874d7
     <collision name='collision'>
       <origin xyz="-0.3 0 0" rpy=" 0 0 1.57079"/>
@@ -153,5 +149,4 @@
         </geometry>
     </collision>
-<<<<<<< HEAD
     <visual>
       <origin xyz=" -0.3 0 0.0" rpy="0 0 1.57079"/>
@@ -159,11 +154,4 @@
         <mesh filename="package://ssabot/meshes/meshes/dumper_bin.dae" scale="0.013 0.013 0.013"/>
       </geometry>
-=======
-    <visual >
-      <origin xyz=" -0.3 0 0.0" rpy="0 0 1.57079"/>
-        <geometry>
-          <mesh filename="package://ssabot/meshes/meshes/dumper_bin.dae" scale="0.013 0.013 0.013"/>
-        </geometry>
->>>>>>> d2d46bd033c6114a82d2ed123778a13e47a874d7
     </visual>
     <inertial>

File: ssapang_ws/src/ssabot/urdf/turtlebot3_waffle.gazebo.xacro (robot description, xacro)
@@ -76,5 +76,5 @@
       <wheelDiameter>0.066</wheelDiameter>
       <wheelAcceleration>1</wheelAcceleration>
-      <wheelTorque>20</wheelTorque>
+      <wheelTorque>10</wheelTorque>
       <rosDebugLevel>na</rosDebugLevel>
     </plugin>
@@ -140,10 +140,46 @@
     </sensor>
   </gazebo>
-  <gazebo reference="piston_plate">
-    <mu1>1</mu1>
-    <mu2>1</mu2>
-    <kp>1000000.0</kp>
-    <kd>10000.0</kd>
-    <material>Gazebo/FlatBlack</material>
+  <gazebo reference="camera_rgb_frame">
+    <sensor type="depth" name="realsense_R200">
+      <always_on>true</always_on>
+      <visualize>$(arg camera_visual)</visualize>
+      <camera>
+          <horizontal_fov>1.3439</horizontal_fov>
+          <image>
+              <width>1920</width>
+              <height>1080</height>
+              <format>R8G8B8</format>
+          </image>
+          <depth_camera></depth_camera>
+          <clip>
+              <near>0.03</near>
+              <far>100</far>
+          </clip>
+      </camera>
+      <plugin name="camera_controller" filename="libgazebo_ros_openni_kinect.so">
+        <baseline>0.2</baseline>
+        <alwaysOn>true</alwaysOn>
+        <updateRate>30.0</updateRate>
+        <cameraName>camera</cameraName>
+        <frameName>camera_rgb_optical_frame</frameName>
+        <imageTopicName>rgb/image_raw</imageTopicName>
+        <depthImageTopicName>depth/image_raw</depthImageTopicName>
+        <pointCloudTopicName>depth/points</pointCloudTopicName>
+        <cameraInfoTopicName>rgb/camera_info</cameraInfoTopicName>
+        <depthImageCameraInfoTopicName>depth/camera_info</depthImageCameraInfoTopicName>
+        <pointCloudCutoff>0.4</pointCloudCutoff>
+            <hackBaseline>0.07</hackBaseline>
+            <distortionK1>0.0</distortionK1>
+            <distortionK2>0.0</distortionK2>
+            <distortionK3>0.0</distortionK3>
+            <distortionT1>0.0</distortionT1>
+            <distortionT2>0.0</distortionT2>
+        <CxPrime>0.0</CxPrime>
+        <Cx>0.0</Cx>
+        <Cy>0.0</Cy>
+        <focalLength>0</focalLength>
+        <hackBaseline>0</hackBaseline>
+      </plugin>
+    </sensor>
   </gazebo>
 </robot>

File: ssapang_ws/src/ssabot/urdf/turtlebot3_waffle.urdf.xacro (robot description, xacro)
@@ -50,5 +50,5 @@
 	  <origin xyz="-0.05 0 0.14" rpy="0 0 0"/>
       <geometry>
-        <cylinder length="0.03" radius="0.025"/>
+        <cylinder length="0.02" radius="0.005"/>
       </geometry>
       <material name="red"/>
@@ -65,11 +65,11 @@
     <origin xyz="0 0 0" rpy="0 0 0"/>
     <axis xyz="0 0 1"/>
-    <limit effort="30" lower="-0.1" upper="0.02" velocity="0.171"/>
+    <limit effort="30" lower="-0.1" upper="0.1" velocity="0.171"/>
   </joint>
   <link name="piston_link2">
     <visual>
-	  <origin xyz="-0.05 0 0.162" rpy="0 0 0"/>
-      <geometry>
-        <cylinder length="0.025" radius="0.015"/>
+	  <origin xyz="-0.05 0 0.16" rpy="0 0 0"/>
+      <geometry>
+        <cylinder length="0.02" radius="0.01"/>
       </geometry>
       <material name="orange"/>
@@ -87,16 +87,17 @@
   <link name="piston_plate">
     <visual>
-      <origin xyz="-0.05 0 0.16" rpy="0 0 1.57"/>
-      <geometry>
-        <mesh filename="package://ssabot/meshes/piston/untitled1.dae" scale="0.01  0.01  0.01"/>
+      <origin xyz="-0.05 0 0.17" rpy="0 0 1.57"/>
+      <geometry>
+        <mesh filename="package://ssabot/meshes/piston/piston_plate.dae" scale="0.015 0.015 0.015"/>
       </geometry>
       <material name="dark"/>
     </visual>
     <collision>
-      <origin xyz="-0.05 0 0.16" rpy="0 0 1.57"/>
-      <geometry>
-        <mesh filename="package://ssabot/meshes/piston/untitled1.dae" scale="0.01  0.01 0.01"/>
-      </geometry>
-    </collision>
+      <origin xyz="-0.05 0 0.17" rpy="0 0 1.57"/>
+      <geometry>
+        <mesh filename="package://ssabot/meshes/piston/piston_plate.dae" scale="0.015 0.015 0.015"/>
+      </geometry>
+    </collision>
+<!--
     <inertial>
       <mass value="0.114" />
@@ -105,5 +106,5 @@
                iyy="0.001" iyz="0.0"
                izz="0.001" />
-    </inertial>
+    </inertial> -->
   </link>
   <transmission name="waffle_tran">
@@ -247,3 +248,54 @@
     </inertial>
   </link>
+  <joint name="camera_joint" type="fixed">
+    <origin xyz="0.064 -0.065 0.094" rpy="0 0 0"/>
+    <parent link="base_link"/>
+    <child link="camera_link"/>
+  </joint>
+  <link name="camera_link">
+    <visual>
+     <origin xyz="0 0 0" rpy="1.57 0 1.57"/>
+      <geometry>
+       <mesh filename="package://ssabot/meshes/sensors/r200.dae" />
+      </geometry>
+    </visual>
+    <collision>
+      <origin xyz="0.003 0.065 0.007" rpy="0 0 0"/>
+      <geometry>
+        <box size="0.012 0.132 0.020"/>
+      </geometry>
+    </collision>
+    <!-- This inertial field needs doesn't contain reliable data!! -->
+<!--   <inertial>
+      <mass value="0.564" />
+      <origin xyz="0 0 0" />
+      <inertia ixx="0.003881243" ixy="0.0" ixz="0.0"
+               iyy="0.000498940" iyz="0.0"
+               izz="0.003879257" />
+    </inertial>-->
+  </link>
+  <joint name="camera_rgb_joint" type="fixed">
+    <origin xyz="${r200_cam_rgb_px} ${r200_cam_rgb_py} ${r200_cam_rgb_pz}" rpy="0 0 0"/>
+    <parent link="camera_link"/>
+    <child link="camera_rgb_frame"/>
+  </joint>
+  <link name="camera_rgb_frame"/>
+  <joint name="camera_rgb_optical_joint" type="fixed">
+    <origin xyz="0 0 0" rpy="-1.57 0 -1.57"/>
+    <parent link="camera_rgb_frame"/>
+    <child link="camera_rgb_optical_frame"/>
+  </joint>
+  <link name="camera_rgb_optical_frame"/>
+  <joint name="camera_depth_joint" type="fixed">
+    <origin xyz="${r200_cam_rgb_px} ${r200_cam_rgb_py + r200_cam_depth_offset} ${r200_cam_rgb_pz}" rpy="0 0 0"/>
+    <parent link="camera_link"/>
+    <child link="camera_depth_frame"/>
+  </joint>
+  <link name="camera_depth_frame"/>
+  <joint name="camera_depth_optical_joint" type="fixed">
+    <origin xyz="0 0 0" rpy="-1.57 0 -1.57"/>
+    <parent link="camera_depth_frame"/>
+    <child link="camera_depth_optical_frame"/>
+  </joint>
+  <link name="camera_depth_optical_frame"/>
 </robot>
