Commit message: [modified] control_tower & robot_control

File: ssapang_ws/src/ssabot/urdf/turtlebot3_waffle.urdf.xacro (robot description, xacro)
@@ -48,5 +48,5 @@
     </collision> -->
     <visual>
-	  <origin xyz="-0.05 0 0.14" rpy="0 0 0"/>
+      <origin xyz="-0.05 0 0.14" rpy="0 0 0"/>
       <geometry>
         <cylinder length="0.02" radius="0.005"/>
@@ -69,5 +69,5 @@
   <link name="piston_link2">
     <visual>
-	  <origin xyz="-0.05 0 0.16" rpy="0 0 0"/>
+      <origin xyz="-0.05 0 0.16" rpy="0 0 0"/>
       <geometry>
         <cylinder length="0.02" radius="0.01"/>

Commit message: [modified] ssapang_map

File: ssapang_ws/src/ssabot/urdf/turtlebot3_waffle.urdf.xacro (robot description, xacro)
@@ -48,5 +48,5 @@
     </collision> -->
     <visual>
-	  <origin xyz="-0.05 0 0.14" rpy="0 0 0"/>
+	  <origin xyz="-0.05 0 0.12" rpy="0 0 0"/>
       <geometry>
         <cylinder length="0.03" radius="0.025"/>
@@ -65,11 +65,11 @@
     <origin xyz="0 0 0" rpy="0 0 0"/>
     <axis xyz="0 0 1"/>
-    <limit effort="30" lower="-0.1" upper="0.02" velocity="0.171"/>
+    <limit effort="30" lower="-0.1" upper="0.05" velocity="0.171"/>
   </joint>
   <link name="piston_link2">
     <visual>
-	  <origin xyz="-0.05 0 0.162" rpy="0 0 0"/>
-      <geometry>
-        <cylinder length="0.025" radius="0.015"/>
+	  <origin xyz="-0.05 0 0.08" rpy="0 0 0"/>
+      <geometry>
+        <cylinder length="0.08" radius="0.015"/>
       </geometry>
       <material name="orange"/>
@@ -87,14 +87,14 @@
   <link name="piston_plate">
     <visual>
-      <origin xyz="-0.05 0 0.16" rpy="0 0 1.57"/>
-      <geometry>
-        <mesh filename="package://ssabot/meshes/piston/untitled1.dae" scale="0.01  0.01  0.01"/>
-      </geometry>
-      <material name="dark"/>
-    </visual>
-    <collision>
-      <origin xyz="-0.05 0 0.16" rpy="0 0 1.57"/>
-      <geometry>
-        <mesh filename="package://ssabot/meshes/piston/untitled1.dae" scale="0.01  0.01 0.01"/>
+      <origin xyz="0.0 0 0.1" rpy="0 0 1.57"/>
+      <geometry>
+        <mesh filename="package://ssabot/meshes/piston/fix_plate.dae" scale="0.01  0.01  0.01"/>
+      </geometry>
+      <material name="dark"/>
+    </visual>
+    <collision>
+      <origin xyz="0 0 0.1" rpy="0 0 1.57"/>
+      <geometry>
+        <mesh filename="package://ssabot/meshes/piston/fix_plate.dae" scale="0.01  0.01 0.01"/>
       </geometry>
     </collision>

Commit message: [modified] ssapang_map

File: ssapang_ws/src/ssabot/urdf/turtlebot3_waffle.urdf.xacro (robot description, xacro)
@@ -65,5 +65,5 @@
     <origin xyz="0 0 0" rpy="0 0 0"/>
     <axis xyz="0 0 1"/>
-    <limit effort="30" lower="-0.1" upper="0.05" velocity="0.171"/>
+    <limit effort="30" lower="-0.1" upper="0.08" velocity="0.171"/>
   </joint>
   <link name="piston_link2">
