Commit message: [Add] push_robot.urdf and qr_tracing.py

File: ssapang_ws/src/ssabot/urdf/push_robot.urdf.xacro (robot description, xacro)
@@ -1,10 +1,14 @@
 <?xml version="1.0" ?>
-<robot name="turtlebot3_waffle" xmlns:xacro="http://ros.org/wiki/xacro">
-  <xacro:include filename="$(find ssabot)/urdf/common_properties.xacro"/>
+<robot name="push_robot" xmlns:xacro="http://ros.org/wiki/xacro">
+  <!-- <xacro:include filename="$(find ssabot)/urdf/common_properties.xacro"/> -->
+  <xacro:include filename="$(find ssabot)/urdf/push_robot.gazebo.xacro" />
+  <material name="black">
+    <color rgba="0.0 0.0 0.0 1.0"/>
+  </material>
   <link name="base_footprint"/>
   <joint name="base_joint" type="fixed">
     <parent link="base_footprint"/>
     <child link="base_link" />
-    <origin xyz="0 0 0" rpy="0 0 0"/>
+    <origin xyz="0 0 0.5" rpy="0 0 0"/>
   </joint>
   <link name="base_link">
@@ -12,12 +16,13 @@
       <origin xyz="0 0 0.05" rpy="0 0 0"/>
       <geometry>
-        <box size="0.1 0.1 0.1"/>
-      </geometry>
-      <material name="light_black"/>
+        <!-- <box size="0.1 0.1 0.1"/> -->
+        <box size="0.5 0.5 0.01"/>
+      </geometry>
     </visual>
     <collision>
       <origin xyz="0 0 0.05" rpy="0 0 0"/>
       <geometry>
-        <box size="0.1 0.1 0.1"/>
+        <!-- <box size="0.1 0.1 0.1"/> -->
+        <box size="0.5 0.5 0.01"/>
       </geometry>
     </collision>
@@ -30,50 +35,80 @@
     </inertial>
   </link>
-  <joint name="virtual_joint1" type="fixed">
+  <joint name="virtual_joint1" type="prismatic">
     <parent link="base_link"/>
     <child link="virtual_link1"/>
-    <origin xyz="0 0 0.2" rpy="0 0 0"/>
+    <origin xyz="0 0 0" rpy="0 0 0"/>
+    <axis xyz="0 1 0"/>
+    <limit effort="30" lower="-0.3" upper="0.3" velocity="0.171"/>
   </joint>
   <link name="virtual_link1">
-    <collision>
-      <origin xyz="0 0 0.05" rpy="0 0 0"/>
-      <geometry>
-          <box size="0.1 0.1 0.1"/>
-      </geometry>
-    </collision>
-    <visual>
-      <origin xyz="0 0 0.05" rpy="0 0 0"/>
-      <geometry>
-          <box size="0.1 0.1 0.1"/>
-      </geometry>
-      <material name="red"/>
-    </visual>
-    <inertial>
-      <origin xyz="0 0 0" rpy="0 0 0"/>
-      <mass value="1.3729096e+00"/>
-      <inertia ixx="8.7002718e-03" ixy="-4.7576583e-05" ixz="1.1160499e-04"
-               iyy="8.6195418e-03" iyz="-3.5422299e-06"
-               izz="1.4612727e-02" />
-    </inertial>
-  </link>
-  <joint name="virtual_joint2" type="fixed">
+    <visual>
+      <origin xyz="0 0 0.5" rpy="0 0 0"/>
+      <geometry>
+        <cylinder length="1" radius="0.01"/>
+      </geometry>
+    </visual>
+    <!-- <collision>
+      <origin xyz="0 0 0.3" rpy="0 0 0"/>
+      <geometry>
+          <box size="0.1 0.1 0.1"/>
+      </geometry>
+    </collision> -->
+    <inertial>
+      <origin xyz="0 0 0" rpy="0 0 0"/>
+      <mass value="1.3729096e+00"/>
+      <inertia ixx="8.7002718e-03" ixy="-4.7576583e-05" ixz="1.1160499e-04"
+               iyy="8.6195418e-03" iyz="-3.5422299e-06"
+               izz="1.4612727e-02" />
+    </inertial>
+  </link>
+  <joint name="virtual_joint2" type="prismatic">
     <parent link="virtual_link1"/>
     <child link="virtual_link2"/>
-    <origin xyz="0 0 1" rpy="0 0 0"/>
+    <origin xyz="0 0 0" rpy="0 0 0"/>
+    <axis xyz="0 0 1"/>
+    <limit effort="30" lower="-0.001" upper="0.001" velocity="0.171"/>
   </joint>
   <link name="virtual_link2">
-    <collision>
-      <origin xyz="0 0 0.05" rpy="0 0 0"/>
-      <geometry>
-          <box size="0.1 0.1 0.1"/>
-      </geometry>
-    </collision>
-    <visual>
-      <origin xyz="0 0 0.05" rpy="0 0 0"/>
-      <geometry>
-          <box size="0.1 0.1 0.1"/>
-      </geometry>
-      <material name="red"/>
-    </visual>
+    <visual>
+      <origin xyz="0 0 0" rpy="-1.57 0 0"/>
+      <geometry>
+        <cylinder length="1" radius="0.01"/>
+      </geometry>
+    </visual>
+    <!-- <collision>
+      <origin xyz="0 0.1 0" rpy="0 0 0"/>
+      <geometry>
+          <box size="0.1 0.1 0.1"/>
+      </geometry>
+    </collision> -->
+    <inertial>
+      <origin xyz="0 0 0" rpy="0 0 0"/>
+      <mass value="1.3729096e+00"/>
+      <inertia ixx="8.7002718e-03" ixy="-4.7576583e-05" ixz="1.1160499e-04"
+               iyy="8.6195418e-03" iyz="-3.5422299e-06"
+               izz="1.4612727e-02" />
+    </inertial>
+  </link>
+  <joint name="virtual_joint3" type="prismatic">
+    <parent link="virtual_link2"/>
+    <child link="virtual_link3"/>
+    <origin xyz="0 0 0" rpy="0 0 0"/>
+    <axis xyz="0 1 0"/>
+    <limit effort="30" lower="-0.001" upper="0.001" velocity="0.171"/>
+  </joint>
+  <link name="virtual_link3">
+    <visual>
+      <origin xyz="0 0 0" rpy="0 0 0"/>
+      <geometry>
+        <box size="0.1 0.1 0.1"/>
+      </geometry>
+    </visual>
+    <!-- <collision>
+      <origin xyz="0 0 0.05" rpy="0 0 0"/>
+      <geometry>
+          <box size="0.1 0.1 0.1"/>
+      </geometry>
+    </collision> -->
     <inertial>
       <origin xyz="0 0 0" rpy="0 0 0"/>
@@ -85,57 +120,70 @@
   </link>
   <joint name="push_joint1" type="fixed">
-    <parent link="virtual_link2"/>
+    <parent link="virtual_link3"/>
     <child link="push_link1"/>
-    <origin xyz="0 0 1" rpy="0 0 0"/>
+    <origin xyz="0 0 0" rpy="0 0 0"/>
   </joint>
   <link name="push_link1">
-    <collision>
-      <origin xyz="0 0 0.05" rpy="0 0 0"/>
-      <geometry>
-          <box size="0.1 0.1 0.1"/>
-      </geometry>
-    </collision>
-    <visual>
-      <origin xyz="0 0 0.05" rpy="0 0 0"/>
-      <geometry>
-          <box size="0.1 0.1 0.1"/>
-      </geometry>
-      <material name="red"/>
-    </visual>
-    <inertial>
-      <origin xyz="0 0 0" rpy="0 0 0"/>
-      <mass value="1.3729096e+00"/>
-      <inertia ixx="8.7002718e-03" ixy="-4.7576583e-05" ixz="1.1160499e-04"
-               iyy="8.6195418e-03" iyz="-3.5422299e-06"
-               izz="1.4612727e-02" />
-    </inertial>
-  </link>
-  <joint name="push_joint2" type="fixed">
+    <visual>
+      <origin xyz="0 0 0" rpy="0 1.57 0"/>
+      <geometry>
+        <cylinder length="0.2" radius="0.05"/>
+      </geometry>
+    </visual>
+    <!-- <collision>
+      <origin xyz="0 0 0.05" rpy="0 0 0"/>
+      <geometry>
+          <box size="0.1 0.1 0.1"/>
+      </geometry>
+    </collision> -->
+    <inertial>
+      <origin xyz="0 0 0" rpy="0 0 0"/>
+      <mass value="1.3729096e+00"/>
+      <inertia ixx="8.7002718e-03" ixy="-4.7576583e-05" ixz="1.1160499e-04"
+               iyy="8.6195418e-03" iyz="-3.5422299e-06"
+               izz="1.4612727e-02" />
+    </inertial>
+  </link>
+  <joint name="push_joint2" type="prismatic">
     <parent link="push_link1"/>
     <child link="push_link2"/>
-    <origin xyz="0 0 1" rpy="0 0 0"/>
+    <origin xyz="0 0 0" rpy="0 0 0"/>
+    <axis xyz="1 0 0"/>
+    <limit effort="30" lower="-0.001" upper="0.001" velocity="0.171"/>
   </joint>
   <link name="push_link2">
-    <collision>
-      <origin xyz="0 0 0.05" rpy="0 0 0"/>
-      <geometry>
-          <box size="0.1 0.1 0.1"/>
-      </geometry>
-    </collision>
-    <visual>
-      <origin xyz="0 0 0.05" rpy="0 0 0"/>
-      <geometry>
-          <box size="0.1 0.1 0.1"/>
-      </geometry>
-      <material name="red"/>
-    </visual>
-    <inertial>
-      <origin xyz="0 0 0" rpy="0 0 0"/>
-      <mass value="1.3729096e+00"/>
-      <inertia ixx="8.7002718e-03" ixy="-4.7576583e-05" ixz="1.1160499e-04"
-               iyy="8.6195418e-03" iyz="-3.5422299e-06"
-               izz="1.4612727e-02" />
-    </inertial>
-  </link>
+    <visual>
+      <origin xyz="0 0 0" rpy="0 1.57 0"/>
+      <geometry>
+        <cylinder length="0.1" radius="0.1"/>
+      </geometry>
+    </visual>
+    <!-- <collision>
+      <origin xyz="0 0 0" rpy="0 0 0"/>
+      <geometry>
+          <box size="0.1 0.1 0.1"/>
+      </geometry>
+    </collision> -->
+    <inertial>
+      <origin xyz="0 0 0" rpy="0 0 0"/>
+      <mass value="1.3729096e+00"/>
+      <inertia ixx="8.7002718e-03" ixy="-4.7576583e-05" ixz="1.1160499e-04"
+               iyy="8.6195418e-03" iyz="-3.5422299e-06"
+               izz="1.4612727e-02" />
+    </inertial>
+  </link>
+  <transmission name="actuator1">
+    <type>transmission_interface/SimpleTransmission</type>
+    <joint name="virtual_joint1">
+      <hardwareInterface>hardware_interface/EffortJointInterface</hardwareInterface>
+    </joint>
+    <!-- <joint name="virtual_joint3">
+      <hardwareInterface>hardware_interface/EffortJointInterface</hardwareInterface>
+    </joint> -->
+    <actuator name="push_motor1">
+      <hardwareInterface>hardware_interface/EffortJointInterface</hardwareInterface>
+      <mechanicalReduction>1</mechanicalReduction>
+    </actuator>
+  </transmission>
   <!--  -->
   <!-- <link name="piston_link2">

Commit message: [Edit] change push_robot effort

File: ssapang_ws/src/ssabot/urdf/push_robot.urdf.xacro (robot description, xacro)
@@ -40,5 +40,5 @@
     <origin xyz="0 0 0.05" rpy="0 0 0"/>
     <axis xyz="0 1 0"/>
-    <limit effort="5" lower="-0.5" upper="0.5" velocity="0.171"/>
+    <limit effort="0.01" lower="-0.5" upper="0.5" velocity="0.0001"/>
   </joint>
   <link name="base_link2">
@@ -94,5 +94,5 @@
     <origin xyz="0 0 0.55" rpy="0 0 0"/>
     <axis xyz="0 0 1"/>
-    <limit effort="5" lower="-0.5" upper="0.5" velocity="0.171"/>
+    <limit effort="0.01" lower="-0.5" upper="0.5" velocity="0.0001"/>
   </joint>
   <link name="virtual_link2">
@@ -122,5 +122,5 @@
     <origin xyz="0 0 0" rpy="0 0 0"/>
     <axis xyz="0 0 1"/>
-    <limit effort="5" lower="-0.5" upper="0.5" velocity="0.171"/>
+    <limit effort="0.01" lower="-0.5" upper="0.5" velocity="0.0001"/>
   </joint>
   <link name="push_link1">
@@ -150,5 +150,5 @@
     <origin xyz="0 0 0" rpy="0 0 0"/>
     <axis xyz="1 0 0"/>
-    <limit effort="30" lower="-0.1" upper="0.1" velocity="0.171"/>
+    <limit effort="0.001" lower="-0.1" upper="0.1" velocity="0.0001"/>
   </joint>
   <link name="push_link2">

Commit message: [Add] add wall to push_robot

File: ssapang_ws/src/ssabot/urdf/push_robot.urdf.xacro (robot description, xacro)
@@ -6,28 +6,27 @@
     <color rgba="0.0 0.0 0.0 1.0"/>
   </material>
-  <link name="base_footprint"/>
+  <link name="world"/>
   <joint name="base_joint" type="fixed">
-    <parent link="base_footprint"/>
-    <child link="base_link1" />
-    <origin xyz="0 0 0" rpy="0 0 0"/>
-  </joint>
-  <link name="base_link1">
-    <visual>
-      <origin xyz="0 0 0.05" rpy="0 0 0"/>
-      <geometry>
-        <!-- <box size="0.1 0.1 0.1"/> -->
-        <box size="0.5 1 0.01"/>
+    <parent link="world"/>
+    <child link="base_link" />
+    <origin xyz="0 0 -0.5" rpy="0 0 0"/>
+  </joint>
+  <link name="base_link">
+    <visual>
+      <origin xyz="0 0 0" rpy="0 0 1.57"/>
+      <geometry>
+        <mesh filename="package://ssabot/meshes/wall.dae" scale="1 1 1"/>
+        <!-- <box size="0.5 1 0.01"/> -->
       </geometry>
     </visual>
     <collision>
-      <origin xyz="0 0 0.05" rpy="0 0 0"/>
-      <geometry>
-        <!-- <box size="0.1 0.1 0.1"/> -->
-        <box size="0.5 1 0.01"/>
+      <origin xyz="0 0 0.2" rpy="0 0 1.57"/>
+      <geometry>
+        <mesh filename="package://ssabot/meshes/wall.dae" scale="1 1 1"/>
       </geometry>
     </collision>
     <inertial>
       <origin xyz="0 0 0" rpy="0 0 0"/>
-      <mass value="1.3729096e+01"/>
+      <mass value="1.3729096e+02"/>
       <inertia ixx="8.7002718e-03" ixy="-4.7576583e-05" ixz="1.1160499e-04"
                iyy="8.6195418e-03" iyz="-3.5422299e-06"
@@ -36,15 +35,15 @@
   </link>
    <joint name="virtual_joint1" type="prismatic">
-    <parent link="base_link1"/>
-    <child link="base_link2"/>
-    <origin xyz="0 0 0.05" rpy="0 0 0"/>
+    <parent link="base_link"/>
+    <child link="virtual_link1"/>
+    <origin xyz="0 0 1" rpy="0 0 0"/>
     <axis xyz="0 1 0"/>
-    <limit effort="0.01" lower="-0.5" upper="0.5" velocity="0.0001"/>
-  </joint>
-  <link name="base_link2">
-    <visual>
-      <origin xyz="0 0 0.05" rpy="0 0 0"/>
-      <geometry>
-        <box size="0.1 0.1 0.1"/>
+    <limit effort="0.03" lower="-0.5" upper="0.5" velocity="0.0001"/>
+  </joint>
+  <link name="virtual_link1">
+    <visual>
+      <origin xyz="0 0 0" rpy="0 0 0"/>
+      <geometry>
+        <cylinder length="1.8" radius="0.05"/>
       </geometry>
     </visual>
@@ -63,36 +62,10 @@
     </inertial>
   </link>
-  <joint name="fixed_joint" type="fixed">
-    <parent link="base_link2"/>
-    <child link="virtual_link1"/>
-    <origin xyz="0 0 0.5" rpy="0 0 0"/>
-  </joint>
-  <link name="virtual_link1">
-    <visual>
-      <origin xyz="0 0 0" rpy="0 0 0"/>
-      <geometry>
-        <cylinder length="1" radius="0.01"/>
-      </geometry>
-    </visual>
-    <!-- <collision>
-      <origin xyz="0 0 0.3" rpy="0 0 0"/>
-      <geometry>
-          <box size="0.1 0.1 0.1"/>
-      </geometry>
-    </collision> -->
-    <inertial>
-      <origin xyz="0 0 0" rpy="0 0 0"/>
-      <mass value="1.3729096e-05"/>
-      <inertia ixx="8.7002718e-03" ixy="-4.7576583e-05" ixz="1.1160499e-04"
-               iyy="8.6195418e-03" iyz="-3.5422299e-06"
-               izz="1.4612727e-02" />
-    </inertial>
-  </link>
   <joint name="virtual_joint2" type="prismatic">
-    <parent link="base_link1"/>
+    <parent link="base_link"/>
     <child link="virtual_link2"/>
-    <origin xyz="0 0 0.55" rpy="0 0 0"/>
+    <origin xyz="0 0 1" rpy="0 0 0"/>
     <axis xyz="0 0 1"/>
-    <limit effort="0.01" lower="-0.5" upper="0.5" velocity="0.0001"/>
+    <limit effort="0.03" lower="-0.5" upper="0.5" velocity="0.0001"/>
   </joint>
   <link name="virtual_link2">
@@ -100,5 +73,5 @@
       <origin xyz="0 0 0" rpy="-1.57 0 0"/>
       <geometry>
-        <cylinder length="1" radius="0.01"/>
+        <cylinder length="1.8" radius="0.05"/>
       </geometry>
     </visual>
@@ -122,5 +95,5 @@
     <origin xyz="0 0 0" rpy="0 0 0"/>
     <axis xyz="0 0 1"/>
-    <limit effort="0.01" lower="-0.5" upper="0.5" velocity="0.0001"/>
+    <limit effort="0.03" lower="-0.5" upper="0.5" velocity="0.0001"/>
   </joint>
   <link name="push_link1">
@@ -128,5 +101,5 @@
       <origin xyz="0 0 0" rpy="0 1.57 0"/>
       <geometry>
-        <cylinder length="0.2" radius="0.05"/>
+        <cylinder length="0.2" radius="0.2"/>
       </geometry>
     </visual>
@@ -156,13 +129,13 @@
       <origin xyz="0 0 0" rpy="0 1.57 0"/>
       <geometry>
-        <cylinder length="0.1" radius="0.1"/>
-      </geometry>
-    </visual>
-    <!-- <collision>
-      <origin xyz="0 0 0" rpy="0 0 0"/>
-      <geometry>
-          <box size="0.1 0.1 0.1"/>
-      </geometry>
-    </collision> -->
+        <cylinder length="0.4" radius="0.1"/>
+      </geometry>
+    </visual>
+    <collision>
+      <origin xyz="0 0 0" rpy="0 1.57 0"/>
+      <geometry>
+        <cylinder length="0.4" radius="0.1"/>
+      </geometry>
+    </collision>
     <inertial>
       <origin xyz="0 0 0" rpy="0 0 0"/>

Commit message: [Add] spawn multiple shelves and push_robot

File: ssapang_ws/src/ssabot/urdf/push_robot.urdf.xacro (robot description, xacro)
@@ -123,5 +123,5 @@
     <origin xyz="0 0 0" rpy="0 0 0"/>
     <axis xyz="1 0 0"/>
-    <limit effort="50" lower="-0.3" upper="0.3" velocity="0.001"/>
+    <limit effort="50" lower="-0.4" upper="0.4" velocity="0.001"/>
   </joint>
   <link name="push_link2">
@@ -129,5 +129,5 @@
       <origin xyz="0 0 0" rpy="0 1.57 0"/>
       <geometry>
-        <cylinder length="0.4" radius="0.1"/>
+        <cylinder length="0.2" radius="0.1"/>
       </geometry>
     </visual>
@@ -135,5 +135,5 @@
       <origin xyz="0 0 0" rpy="0 1.57 0"/>
       <geometry>
-        <cylinder length="0.4" radius="0.1"/>
+        <cylinder length="0.2" radius="0.1"/>
       </geometry>
     </collision>

Commit message: [Edit] resize push_robot cylinder length

File: ssapang_ws/src/ssabot/urdf/push_robot.urdf.xacro (robot description, xacro)
@@ -101,5 +101,5 @@
       <origin xyz="0 0 0" rpy="0 1.57 0"/>
       <geometry>
-        <cylinder length="0.2" radius="0.2"/>
+        <cylinder length="0.18" radius="0.2"/>
       </geometry>
     </visual>
@@ -129,5 +129,5 @@
       <origin xyz="0 0 0" rpy="0 1.57 0"/>
       <geometry>
-        <cylinder length="0.2" radius="0.1"/>
+        <cylinder length="0.18" radius="0.1"/>
       </geometry>
     </visual>
@@ -135,5 +135,5 @@
       <origin xyz="0 0 0" rpy="0 1.57 0"/>
       <geometry>
-        <cylinder length="0.2" radius="0.1"/>
+        <cylinder length="0.18" radius="0.1"/>
       </geometry>
     </collision>
