Commit message: [Add] Burger dump robot

File: ssapang_ws/src/ssabot/urdf/push_robot.urdf.xacro (robot description, xacro)
@@ -76,10 +76,4 @@
       </geometry>
     </visual>
-    <!-- <collision>
-      <origin xyz="0 0.1 0" rpy="0 0 0"/>
-      <geometry>
-          <box size="0.1 0.1 0.1"/>
-      </geometry>
-    </collision> -->
     <inertial>
       <origin xyz="0 0 0" rpy="-1.57 0 0"/>
@@ -123,5 +117,5 @@
     <origin xyz="0 0 0" rpy="0 0 0"/>
     <axis xyz="1 0 0"/>
-    <limit effort="50" lower="-0.4" upper="0.4" velocity="0.001"/>
+    <limit effort="50" lower="-1" upper="1" velocity="0.01"/>
   </joint>
   <link name="push_link2">
@@ -135,5 +129,5 @@
       <origin xyz="0 0 0" rpy="0 1.57 0"/>
       <geometry>
-        <cylinder length="0.18" radius="0.1"/>
+        <cylinder length="0.18" radius="0.15"/>
       </geometry>
     </collision>

File: ssapang_ws/src/ssabot/urdf/turtlebot3_burger.gazebo.xacro (robot description, xacro)
@@ -4,24 +4,38 @@
   <xacro:arg name="imu_visual"   default="false"/>
   <xacro:arg name="camera_visual" default="false"/>
+  <transmission name="dump_bin_actuator">
+          <type>transmission_interface/SimpleTransmission</type>
+          <joint name="dump_joint">
+              <hardwareInterface>hardware_interface/EffortJointInterface</hardwareInterface>
+          </joint>
+          <actuator name="dump_motor">
+              <hardwareInterface>hardware_interface/EffortJointInterface</hardwareInterface>
+              <mechanicalReduction>1</mechanicalReduction>
+          </actuator>
+    </transmission>
+  <gazebo>
+    <plugin name="gazebo_ros_control" filename="libgazebo_ros_control.so">
+    </plugin>
+  </gazebo>
   <gazebo reference="base_link">
     <material>Gazebo/DarkGrey</material>
   </gazebo>
   <gazebo reference="wheel_left_link">
-    <mu1>0.1</mu1>
-    <mu2>0.1</mu2>
-    <kp>500000.0</kp>
-    <kd>10.0</kd>
+    <mu1>0.2</mu1>
+    <mu2>0.2</mu2>
+    <kp>1000000.0</kp>
+    <kd>20.0</kd>
     <minDepth>0.001</minDepth>
-    <maxVel>0.1</maxVel>
+    <maxVel>0.2</maxVel>
     <fdir1>1 0 0</fdir1>
     <material>Gazebo/FlatBlack</material>
   </gazebo>
   <gazebo reference="wheel_right_link">
-    <mu1>0.1</mu1>
-    <mu2>0.1</mu2>
-    <kp>500000.0</kp>
-    <kd>10.0</kd>
+    <mu1>0.2</mu1>
+    <mu2>0.2</mu2>
+    <kp>1000000.0</kp>
+    <kd>20.0</kd>
     <minDepth>0.001</minDepth>
-    <maxVel>0.1</maxVel>
+    <maxVel>0.2</maxVel>
     <fdir1>1 0 0</fdir1>
     <material>Gazebo/FlatBlack</material>
@@ -58,8 +72,8 @@
       <leftJoint>wheel_left_joint</leftJoint>
       <rightJoint>wheel_right_joint</rightJoint>
-      <wheelSeparation>0.160</wheelSeparation>
-      <wheelDiameter>0.066</wheelDiameter>
+      <wheelSeparation>0.320</wheelSeparation>
+      <wheelDiameter>0.132</wheelDiameter>
       <wheelAcceleration>1</wheelAcceleration>
-      <wheelTorque>10</wheelTorque>
+      <wheelTorque>15</wheelTorque>
       <rosDebugLevel>na</rosDebugLevel>
     </plugin>
@@ -125,6 +139,10 @@
     </sensor>
   </gazebo>
+  <!-- dump_box -->
+  <gazebo reference="dump_box_visual">
+    <material>Gazebo/Orange</material>
+  </gazebo>
   <!-- add waffle_pi camera -->
-  <gazebo reference="camera_rgb_frame">
+  <!-- <gazebo reference="camera_rgb_frame">
     <sensor type="camera" name="Pi Camera">
       <always_on>true</always_on>
@@ -135,6 +153,4 @@
               <width>640</width>
               <height>480</height>
-              <!-- <width>480</width> -->
-              <!-- <height>640</height> -->
               <format>R8G8B8</format>
           </image>
@@ -159,7 +175,7 @@
       </plugin>
     </sensor>
-  </gazebo>
+  </gazebo> -->
   <!-- add second camera -->
-  <gazebo reference="camera_rgb_frame2">
+  <!-- <gazebo reference="camera_rgb_frame2">
     <sensor type="camera" name="Pi Camera">
       <always_on>true</always_on>
@@ -168,6 +184,4 @@
           <horizontal_fov>1.085595</horizontal_fov>
           <image>
-              <!-- <width>640</width> -->
-              <!-- <height>480</height> -->
               <width>480</width>
               <height>640</height>
@@ -194,4 +208,4 @@
       </plugin>
     </sensor>
-  </gazebo>
+  </gazebo> -->
 </robot>

File: ssapang_ws/src/ssabot/urdf/turtlebot3_burger.urdf.xacro (robot description, xacro)
@@ -7,18 +7,18 @@
     <parent link="base_footprint"/>
     <child link="base_link"/>
-    <origin xyz="0.0 0.0 0.010" rpy="0 0 0"/>
+    <origin xyz="0.0 0.0 0.020" rpy="0 0 0"/>
   </joint>
   <link name="base_link">
     <visual>
-      <origin xyz="-0.032 0 0.0" rpy="0 0 0"/>
+      <origin xyz="-0.064 0 0.0" rpy="0 0 0"/>
       <geometry>
-        <mesh filename="package://ssabot/meshes/bases/burger_base.stl" scale="0.001 0.001 0.001"/>
+        <mesh filename="package://ssabot/meshes/bases/burger_base.stl" scale="0.002 0.002 0.002"/>
       </geometry>
       <material name="light_black"/>
     </visual>
     <collision>
-      <origin xyz="-0.032 0 0.070" rpy="0 0 0"/>
+      <origin xyz="-0.064 0 0.140" rpy="0 0 0"/>
       <geometry>
-        <box size="0.140 0.140 0.143"/>
+        <box size="0.280 0.280 0.286"/>
       </geometry>
     </collision>
@@ -34,5 +34,5 @@
     <parent link="base_link"/>
     <child link="wheel_left_link"/>
-    <origin xyz="0.0 0.08 0.023" rpy="-1.57 0 0"/>
+    <origin xyz="0.0 0.16 0.046" rpy="-1.57 0 0"/>
     <axis xyz="0 0 1"/>
   </joint>
@@ -41,5 +41,5 @@
       <origin xyz="0 0 0" rpy="1.57 0 0"/>
       <geometry>
-        <mesh filename="package://ssabot/meshes/wheels/left_tire.stl" scale="0.001 0.001 0.001"/>
+        <mesh filename="package://ssabot/meshes/wheels/left_tire.stl" scale="0.002 0.002 0.002"/>
       </geometry>
       <material name="dark"/>
@@ -48,19 +48,19 @@
       <origin xyz="0 0 0" rpy="0 0 0"/>
       <geometry>
-        <cylinder length="0.018" radius="0.033"/>
+        <cylinder length="0.036" radius="0.066"/>
       </geometry>
     </collision>
     <inertial>
       <origin xyz="0 0 0" />
-      <mass value="2.8498940e-02" />
-      <inertia ixx="1.1175580e-05" ixy="-4.2369783e-11" ixz="-5.9381719e-09"
-               iyy="1.1192413e-05" iyz="-1.4400107e-11"
-               izz="2.0712558e-05" />
-      </inertial>
+      <mass value="5.6398940e-02" />
+      <inertia ixx="2.1175580e-05" ixy="-8.2369783e-11" ixz="-10.9381719e-09"
+               iyy="2.1192413e-05" iyz="-2.4400107e-11"
+               izz="4.0712558e-05" />
+    </inertial>
   </link>
   <joint name="wheel_right_joint" type="continuous">
     <parent link="base_link"/>
     <child link="wheel_right_link"/>
-    <origin xyz="0.0 -0.080 0.023" rpy="-1.57 0 0"/>
+    <origin xyz="0.0 -0.160 0.046" rpy="-1.57 0 0"/>
     <axis xyz="0 0 1"/>
   </joint>
@@ -69,5 +69,5 @@
       <origin xyz="0 0 0" rpy="1.57 0 0"/>
       <geometry>
-        <mesh filename="package://ssabot/meshes/wheels/right_tire.stl" scale="0.001 0.001 0.001"/>
+        <mesh filename="package://ssabot/meshes/wheels/right_tire.stl" scale="0.002 0.002 0.002"/>
       </geometry>
       <material name="dark"/>
@@ -76,13 +76,13 @@
       <origin xyz="0 0 0" rpy="0 0 0"/>
       <geometry>
-        <cylinder length="0.018" radius="0.033"/>
+        <cylinder length="0.036" radius="0.066"/>
       </geometry>
     </collision>
     <inertial>
       <origin xyz="0 0 0" />
-      <mass value="2.8498940e-02" />
-      <inertia ixx="1.1175580e-05" ixy="-4.2369783e-11" ixz="-5.9381719e-09"
-               iyy="1.1192413e-05" iyz="-1.4400107e-11"
-               izz="2.0712558e-05" />
+      <mass value="5.6398940e-02" />
+      <inertia ixx="2.1175580e-05" ixy="-8.2369783e-11" ixz="-10.9381719e-09"
+               iyy="2.1192413e-05" iyz="-2.4400107e-11"
+               izz="4.0712558e-05" />
       </inertial>
   </link>
@@ -90,19 +90,19 @@
     <parent link="base_link"/>
     <child link="caster_back_link"/>
-    <origin xyz="-0.081 0 -0.004" rpy="-1.57 0 0"/>
+    <origin xyz="-0.162 0 -0.008" rpy="-1.57 0 0"/>
   </joint>
   <link name="caster_back_link">
     <collision>
-      <origin xyz="0 0.001 0" rpy="0 0 0"/>
+      <origin xyz="0 0.002 0" rpy="0 0 0"/>
       <geometry>
-        <box size="0.030 0.009 0.020"/>
+        <box size="0.060 0.018 0.040"/>
       </geometry>
     </collision>
     <inertial>
       <origin xyz="0 0 0" />
-      <mass value="0.005" />
-      <inertia ixx="0.001" ixy="0.0" ixz="0.0"
-               iyy="0.001" iyz="0.0"
-               izz="0.001" />
+      <mass value="0.010" />
+      <inertia ixx="0.002" ixy="0.0" ixz="0.0"
+               iyy="0.002" iyz="0.0"
+               izz="0.002" />
     </inertial>
   </link>
@@ -113,25 +113,47 @@
   </joint>
   <link name="imu_link"/>
-  <joint name="scan_joint" type="fixed">
+  <joint name="dump_joint" type="revolute">
     <parent link="base_link"/>
-    <child link="base_scan"/>
-    <origin xyz="-0.032 0 0.172" rpy="0 0 0"/>
+    <child link="dumper_bin"/>
+    <origin xyz="0.2 0 0.28" rpy="0 0 0"/>
+    <axis xyz="0 1 0"/>
+    <limit effort="1" velocity="1" lower="0" upper="0.6"/>
   </joint>
-  <link name="base_scan">
-    <visual>
-      <origin xyz="0 0 0.0" rpy="0 0 0"/>
-      <geometry>
-        <mesh filename="package://ssabot/meshes/sensors/lds.stl" scale="0.001 0.001 0.001"/>
-      </geometry>
-      <material name="dark"/>
+  <!-- <link name="dumper_bin">
+    <collision name='collision'>
+      <origin xyz="-0.15 0 0" rpy=" 0 0 1.57079"/>
+        <geometry>
+          <box size="0.3 0.3 0.01"/>
+        </geometry>
+    </collision>
+    <visual name='dump_box_visual'>
+      <origin xyz=" -0.15 0 0.0" rpy="0 0 1.57079"/>
+        <geometry>
+          <box size="0.3 0.3 0.01"/>
+        </geometry>
     </visual>
-    <collision>
-      <origin xyz="0.015 0 -0.0065" rpy="0 0 0"/>
-      <geometry>
-        <cylinder length="0.0315" radius="0.055"/>
-      </geometry>
+    <inertial>
+      <mass value="0.0001" />
+      <origin xyz="0 0 0" />
+      <inertia ixx="0.001" ixy="0.0" ixz="0.0"
+               iyy="0.001" iyz="0.0"
+               izz="0.001" />
+    </inertial>
+  </link> -->
+  <link name="dumper_bin">
+    <collision name='collision'>
+      <origin xyz="-0.3 0 0" rpy=" 0 0 1.57079"/>
+        <geometry>
+          <mesh filename="package://ssabot/meshes/meshes/dumper_bin.dae" scale="0.015 0.015 0.015"/>
+        </geometry>
     </collision>
+    <visual name='dump_box_visual'>
+      <origin xyz=" -0.3 0 0.0" rpy="0 0 1.57079"/>
+        <geometry>
+          <mesh filename="package://ssabot/meshes/meshes/dumper_bin.dae" scale="0.015 0.015 0.015"/>
+        </geometry>
+    </visual>
     <inertial>
-      <mass value="0.114" />
+      <mass value="0.001" />
       <origin xyz="0 0 0" />
       <inertia ixx="0.001" ixy="0.0" ixz="0.0"
@@ -140,57 +162,3 @@
     </inertial>
   </link>
-<!-- add waffle_pi camera -->
-  <joint name="camera_joint" type="fixed">
-    <origin xyz="0.073 -0.011 0.084" rpy="0 0 0"/>
-    <!-- <origin xyz="0.073 -0.011 0.084" rpy="0 45 0"/> -->
-    <parent link="base_link"/>
-    <child link="camera_link"/>
-  </joint>
-  <link name="camera_link">
-    <collision>
-      <origin xyz="0.005 0.011 0.013" rpy="0 0 0"/>
-      <geometry>
-        <box size="0.015 0.030 0.027"/>
-      </geometry>
-    </collision>
-  </link>
-  <joint name="camera_rgb_joint" type="fixed">
-    <origin xyz="0.003 0.011 0.009" rpy="0 0 0"/>
-    <parent link="camera_link"/>
-    <child link="camera_rgb_frame"/>
-  </joint>
-  <link name="camera_rgb_frame"/>
-  <joint name="camera_rgb_optical_joint" type="fixed">
-    <origin xyz="0 0 0" rpy="-1.57 0 -1.57"/>
-    <parent link="camera_rgb_frame"/>
-    <child link="camera_rgb_optical_frame"/>
-  </joint>
-  <link name="camera_rgb_optical_frame"/>
-  <!-- add second camera -->
-  <joint name="camera_joint2" type="fixed">
-    <!-- <origin xyz="0.073 -0.011 0.084" rpy="0 0 0"/> -->
-    <origin xyz="0.073 -0.011 1.084" rpy="0 0 0"/>
-    <parent link="base_link"/>
-    <child link="camera_link2"/>
-  </joint>
-  <link name="camera_link2">
-    <collision>
-      <origin xyz="0.005 0.011 0.013" rpy="0 0 0"/>
-      <geometry>
-        <box size="0.015 0.030 0.027"/>
-      </geometry>
-    </collision>
-  </link>
-  <joint name="camera_rgb_joint2" type="fixed">
-    <origin xyz="0.003 0.011 0.009" rpy="0 0 0"/>
-    <parent link="camera_link2"/>
-    <child link="camera_rgb_frame2"/>
-  </joint>
-  <link name="camera_rgb_frame2"/>
-  <joint name="camera_rgb_optical_joint2" type="fixed">
-    <origin xyz="0 0 0" rpy="-1.57 0 -1.57"/>
-    <parent link="camera_rgb_frame2"/>
-    <child link="camera_rgb_optical_frame2"/>
-  </joint>
-  <link name="camera_rgb_optical_frame2"/>
 </robot>

Commit message: [Add] shelf holes

File: ssapang_ws/src/ssabot/urdf/push_robot.urdf.xacro (robot description, xacro)
@@ -117,5 +117,5 @@
     <origin xyz="0 0 0" rpy="0 0 0"/>
     <axis xyz="1 0 0"/>
-    <limit effort="50" lower="-1" upper="1" velocity="0.01"/>
+    <limit effort="60" lower="-1" upper="1" velocity="0.01"/>
   </joint>
   <link name="push_link2">
@@ -123,5 +123,5 @@
       <origin xyz="0 0 0" rpy="0 1.57 0"/>
       <geometry>
-        <cylinder length="0.18" radius="0.1"/>
+        <cylinder length="0.18" radius="0.15"/>
       </geometry>
     </visual>

Commit message: [modified] ssapang_map

File: ssapang_ws/src/ssabot/urdf/push_robot.urdf.xacro (robot description, xacro)
@@ -39,5 +39,5 @@
     <origin xyz="0 0 1" rpy="0 0 0"/>
     <axis xyz="0 1 0"/>
-    <limit effort="0.03" lower="-0.5" upper="0.5" velocity="0.0001"/>
+    <limit effort="0.185" lower="-1" upper="1" velocity="0.001"/>
   </joint>
   <link name="virtual_link1">
@@ -95,5 +95,5 @@
       <origin xyz="0 0 0" rpy="0 1.57 0"/>
       <geometry>
-        <cylinder length="0.18" radius="0.2"/>
+        <cylinder length="0.1" radius="0.2"/>
       </geometry>
     </visual>

Commit message: [Modify]

File: ssapang_ws/src/ssabot/urdf/push_robot.urdf.xacro (robot description, xacro)
@@ -117,5 +117,5 @@
     <origin xyz="0 0 0" rpy="0 0 0"/>
     <axis xyz="1 0 0"/>
-    <limit effort="50" lower="-1" upper="1" velocity="0.01"/>
+    <limit effort="50" lower="-0" upper="0" velocity="0.01"/>
   </joint>
   <link name="push_link2">

File: ssapang_ws/src/ssabot/urdf/turtlebot3_waffle.urdf.xacro (robot description, xacro)
@@ -65,5 +65,5 @@
     <origin xyz="0 0 0" rpy="0 0 0"/>
     <axis xyz="0 0 1"/>
-    <limit effort="30" lower="-0.1" upper="0.07" velocity="0.171"/>
+    <limit effort="30" lower="-0.1" upper="0.08" velocity="0.171"/>
   </joint>
   <link name="piston_link2">
@@ -87,14 +87,14 @@
   <link name="piston_plate">
     <visual>
-      <origin xyz="0.01 0 0.1" rpy="0 0 1.57"/>
-      <geometry>
-        <mesh filename="package://ssabot/meshes/piston/fix_plate.dae" scale="0.011  0.011  0.01"/>
-      </geometry>
-      <material name="dark"/>
-    </visual>
-    <collision>
-      <origin xyz="0.01 0 0.1" rpy="0 0 1.57"/>
-      <geometry>
-        <mesh filename="package://ssabot/meshes/piston/fix_plate.dae" scale="0.011  0.011 0.01"/>
+      <origin xyz="0.001 0 0.1" rpy="0 0 1.57"/>
+      <geometry>
+        <mesh filename="package://ssabot/meshes/piston/fix_plate.dae" scale="0.01  0.01  0.01"/>
+      </geometry>
+      <material name="dark"/>
+    </visual>
+    <collision>
+      <origin xyz="0.001 0 0.1" rpy="0 0 1.57"/>
+      <geometry>
+        <mesh filename="package://ssabot/meshes/piston/fix_plate.dae" scale="0.01  0.01 0.01"/>
       </geometry>
     </collision>
